Commit message: add static positioner link and fix positioner planning group

File: urdf/positioner_macro.xacro (robot description, xacro)
@@ -33,9 +33,9 @@
     </link>
     <link name="${prefix}positioner"/>
+    <link name="${prefix}positioner_static"/>
     <!-- joint list -->
     <joint name="{prefix}rotary_table_top_base" type="fixed">
       <parent link="${prefix}rotary_table_base"/>
       <child link="${prefix}rotary_table_top"/>
-      <axis xyz="0 0 0"/>
       <origin rpy="0.0 0.0 0.0" xyz="0 0 0.1778"/>
     </joint>
@@ -52,4 +52,9 @@
       <child link="${prefix}positioner"/>
     </joint>
+    <joint name="${prefix}positioner_static_joint" type="fixed">
+      <origin rpy="0.0 0.0 0.0" xyz="0 0 0.03175"/>
+      <parent link="${prefix}rotary_table_top"/>
+      <child link="${prefix}positioner_static"/>
+    </joint>
   </xacro:macro>
 </robot>

Commit message: exchange rotary table for Tormach Super Spacer 8 inch

File: urdf/positioner_macro.xacro (robot description, xacro)
@@ -6,5 +6,5 @@
         <visual>
         <geometry>
-          <mesh filename="package://hydra_description/meshes/rotary_table.dae"/>
+          <mesh filename="package://hydra_description/meshes/visual/rotary_table.dae"/>
         </geometry>
         <origin rpy="0.0 0.0 0.0" xyz="0 0 0"/>
@@ -12,5 +12,5 @@
       <collision>
         <geometry>
-          <mesh filename="package://hydra_description/meshes/rotary_table.dae"/>
+          <mesh filename="package://hydra_description/meshes/collision/rotary_table_collision.stl"/>
         </geometry>
         <origin rpy="0.0 0.0 0.0" xyz="0 0 0"/>
@@ -21,5 +21,5 @@
         <visual>
         <geometry>
-          <mesh filename="package://hydra_description/meshes/hydra_positioner.dae"/>
+          <mesh filename="package://hydra_description/meshes/visual/hydra_positioner.dae"/>
         </geometry>
         <origin rpy="0.0 0.0 0.0" xyz="0 0 0"/>
@@ -27,5 +27,5 @@
       <collision>
         <geometry>
-          <mesh filename="package://hydra_description/meshes/hydra_positioner.dae"/>
+          <mesh filename="package://hydra_description/meshes/collision/hydra_positioner_collision.stl"/>
         </geometry>
         <origin rpy="0.0 0.0 0.0" xyz="0 0 0"/>
@@ -38,5 +38,5 @@
       <parent link="${prefix}rotary_table_base"/>
       <child link="${prefix}rotary_table_top"/>
-      <origin rpy="0.0 0.0 0.0" xyz="0 0 0.1778"/>
+      <origin rpy="0.0 0.0 0.0" xyz="0 0 0.183984"/>
     </joint>
     <joint name="${prefix}rotary_table_positioner" type="continuous">

File: urdf/za_typhoon_macro.xacro (robot description, xacro)
@@ -8,5 +8,5 @@
         <visual>
         <geometry>
-          <mesh filename="package://hydra_description/meshes/typhoon_extruder.dae"/>
+          <mesh filename="package://hydra_description/meshes/visual/typhoon_extruder.dae"/>
         </geometry>
         <origin rpy="0.0 0.0 0.0" xyz="0 0 0"/>
@@ -14,5 +14,5 @@
       <collision>
         <geometry>
-          <mesh filename="package://hydra_description/meshes/typhoon_extruder.dae"/>
+          <mesh filename="package://hydra_description/meshes/visual/typhoon_extruder.dae"/>
         </geometry>
         <origin rpy="0.0 0.0 0.0" xyz="0 0 0"/>
