Commit message: switch to new za6 ikfast plugin

File: urdf/za_typhoon_macro.xacro (robot description, xacro)
@@ -22,10 +22,10 @@
       <origin rpy="0.0 0.0 0.0" xyz="0.0 0.0 0.0"/>
     </link>
-    <!-- attach extruder to tool0 -->
+    <!-- attach extruder to flange -->
     <joint name="${prefix}extruder_attach_joint" type="fixed">
-      <parent link="${prefix}tool0"/>
+      <parent link="${prefix}flange"/>
       <child link="${prefix}typhoon_extruder_base"/>
       <axis xyz="0 0 0"/>
-      <origin rpy="0.0 0.0 0.0" xyz="0 0 0"/>
+      <origin rpy="0.0 ${pi/2} 0.0" xyz="0 0 0"/>
     </joint>
     <joint name="${prefix}extruder_extruder_base" type="fixed">
