Commit message: add gazebo tags in hydra urdf

File: urdf/hydra_macro.xacro (robot description, xacro)
@@ -4,4 +4,6 @@
     <xacro:include filename="$(find hydra_description)/urdf/positioner/positioner_macro.xacro"/>
     <xacro:macro name="hydra_macro" params="prefix radius tool:='tool0'">
+        <!-- Is the robot being simulated in gazebo? -->
+        <xacro:arg name="gazebo" default="true" />
         <xacro:za_pedestal_macro prefix="${prefix}rob1_" tool="${tool}"/>
         <xacro:za_pedestal_macro prefix="${prefix}rob2_" tool="${tool}"/>
@@ -29,4 +31,16 @@
             <child  link="${prefix}positioner_stand_base"/>
         </joint>
+        <xacro:if value="$(arg gazebo)">
+            <transmission name="${prefix}hydra_model">
+              <type>hydra_hw/HydraModelInterface</type>
+              <joint name="${prefix}positioner_joint">
+                <role>positioner</role>
+                <hardwareInterface>hydra_hw/HydraModelInterface</hardwareInterface>
+              </joint>
+              <actuator name="${prefix}_motor_positioner_joint">
+                <hardwareInterface>hydra_hw/HydraModelInterface</hardwareInterface>
+              </actuator>
+            </transmission>
+        </xacro:if>
     </xacro:macro>
 </robot>

Commit message: reverse pedestal chain direction

File: urdf/hydra_macro.xacro (robot description, xacro)
@@ -3,17 +3,21 @@
   <xacro:include filename="$(find hydra_description)/urdf/robots/za_pedestal_macro.xacro"/>
   <xacro:macro name="hydra_macro" params="prefix radius tool:='tool0'">
+    <xacro:property name="rob1_base_origin" value="0 -${radius} 0"/>
+    <xacro:property name="rob1_base_rot" value="0 0 ${pi/2}"/>
+    <xacro:property name="rob2_base_origin" value="0 ${radius} 0"/>
+    <xacro:property name="rob2_base_rot" value="0 0 -${pi/2}"/>
     <xacro:za_pedestal_macro prefix="${prefix}rob1_" tool="${tool}"/>
     <xacro:za_pedestal_macro prefix="${prefix}rob2_" tool="${tool}"/>
     <link name="${prefix}hydra_base"/>
     <!-- joint list -->
-    <joint name="${prefix}hydra_base-rob1_pedestal_base" type="fixed">
+    <joint name="${prefix}hydra_base-rob1_base_link" type="fixed">
       <parent link="${prefix}hydra_base"/>
-      <child  link="${prefix}rob1_pedestal_base"/>
-      <origin xyz="0 -${radius}  0" rpy="0 0 ${pi/2}"/>
+      <child  link="${prefix}rob1_base_link"/>
+      <origin xyz="${rob1_base_origin}" rpy="${rob1_base_rot}"/>
     </joint>
-    <joint name="${prefix}hydra_base-rob2_pedestal_base" type="fixed">
+    <joint name="${prefix}hydra_base-rob2_base_link" type="fixed">
       <parent link="${prefix}hydra_base"/>
-      <child  link="${prefix}rob2_pedestal_base"/>
-      <origin xyz="0 ${radius} 0" rpy="0 0 -${pi/2}"/>
+      <child  link="${prefix}rob2_base_link"/>
+      <origin xyz="${rob2_base_origin}" rpy="${rob2_base_rot}"/>
     </joint>
   </xacro:macro>

File: urdf/robots/za_pedestal_macro.xacro (robot description, xacro)
@@ -31,17 +31,17 @@
     </link>
     <link name="${prefix}pedestal_top"/>
-    <joint name="${prefix}pedestal_base-${prefix}pedestal" type="fixed">
-      <origin rpy="0.0 0.0 0.0" xyz="0 0 ${base_height}"/>
-      <parent link="${prefix}pedestal_base"/>
+    <joint name="${prefix}base_link-${prefix}pedestal_top" type="fixed">
+      <parent link="${prefix}base_link"/>
+      <child  link="${prefix}pedestal_top"/>
+    </joint>
+    <joint name="${prefix}pedestal_top-${prefix}pedestal" type="fixed">
+      <origin rpy="0.0 0.0 0.0" xyz="0 0 ${-ped_height}"/>
+      <parent link="${prefix}pedestal_top"/>
       <child  link="${prefix}pedestal"/>
     </joint>
-    <joint name="${prefix}pedestal-${prefix}pedestal_top" type="fixed">
-      <origin rpy="0.0 0.0 0.0" xyz="0 0 ${ped_height}"/>
+    <joint name="${prefix}pedestal-${prefix}pedestal_base" type="fixed">
+      <origin rpy="0.0 0.0 0.0" xyz="0 0 ${-base_height}"/>
       <parent link="${prefix}pedestal"/>
-      <child  link="${prefix}pedestal_top"/>
-    </joint>
-    <joint name="${prefix}pedestal_top-${prefix}base_link" type="fixed">
-      <parent link="${prefix}pedestal_top"/>
-      <child  link="${prefix}base_link"/>
+      <child  link="${prefix}pedestal_base"/>
     </joint>
   </xacro:macro>
