Commit message: Add robot and positioner pedestals

File: urdf/hydra.xacro (robot description, xacro)
@@ -2,33 +2,12 @@
 <robot name="hydra" xmlns:xacro="http://www.ros.org/wiki/xacro">
   <xacro:arg name="prefix" default=""/>
-  <xacro:arg name="fixed_tool" default="True"/>
-  <xacro:arg name="radius" default="0.9"/>
+  <xacro:property name="radius" value="0.95" />
+  <xacro:property name="tool" default="typhoon_extruder" />
   <xacro:include filename="$(find hydra_description)/urdf/hydra_macro.xacro"/>
-  <xacro:hydra_macro prefix="$(arg prefix)"/>
-  <!-- 'world' frame: default pose reference frame -->
-  <link name="world" />
-  <joint name="world-$(arg prefix)rob1_base_link" type="fixed">
-    <origin xyz="-${$(arg radius)*sin(pi/6)} -${$(arg radius)*cos(pi/6)}  0" rpy="0 0 ${pi/3}"/>
-    <axis xyz="0 0 1"/>
-    <parent link="world"/>
-    <child link="$(arg prefix)rob1_base_link"/>
-  </joint>
-  <joint name="world-$(arg prefix)rob2_base_link" type="fixed">
-    <origin xyz="${$(arg radius)} 0 0" rpy="0 0 ${pi}"/>
-    <axis xyz="0 0 1"/>
-    <parent link="world"/>
-    <child link="$(arg prefix)rob2_base_link"/>
-  </joint>
-  <joint name="world-$(arg prefix)rob3_base_link" type="fixed">
-    <origin xyz="-${$(arg radius)*sin(pi/6)} ${$(arg radius)*cos(pi/6)} 0" rpy="0 0 -${pi/3}"/>
-    <axis xyz="0 0 1"/>
-    <parent link="world"/>
-    <child link="$(arg prefix)rob3_base_link"/>
-  </joint>
-  <joint name="world-$(arg prefix)rotary_table_base" type="fixed">
-    <origin xyz="0 0 0"/>
-    <axis xyz="0 0 1"/>
-    <parent link="world"/>
-    <child link="$(arg prefix)rotary_table_base"/>
+  <xacro:hydra_macro prefix="$(arg prefix)" radius="${radius}" tool="${tool}"/>
+  <link name="world"/>
+  <joint name="world-$(arg prefix)hydra_base" type="fixed">
+      <parent link="world"/>
+      <child  link="$(arg prefix)hydra_base"/>
   </joint>
 </robot>

File: urdf/hydra_macro.xacro (robot description, xacro)
@@ -1,11 +1,32 @@
 <?xml version="1.0" ?>
 <robot name="hydra" xmlns:xacro="http://www.ros.org/wiki/xacro">
-    <xacro:include filename="$(find hydra_description)/urdf/za_typhoon_macro.xacro"/>
-    <xacro:include filename="$(find hydra_description)/urdf/positioner_macro.xacro"/>
-    <xacro:macro name="hydra_macro" params="prefix">
-        <xacro:za_typhoon_macro prefix="${prefix}rob1_" tool0_trans="0 0 0" tool0_rot="0 ${pi*1} 0"/>
-        <xacro:za_typhoon_macro prefix="${prefix}rob2_" tool0_trans="0 0 0" tool0_rot="0 ${pi*1} 0"/>
-        <xacro:za_typhoon_macro prefix="${prefix}rob3_" tool0_trans="0 0 0" tool0_rot="0 ${pi*1} 0"/>
+    <xacro:include filename="$(find hydra_description)/urdf/robots/za_pedestal_macro.xacro"/>
+    <xacro:include filename="$(find hydra_description)/urdf/positioner/positioner_macro.xacro"/>
+    <xacro:macro name="hydra_macro" params="prefix radius tool:='tool0'">
+        <xacro:za_pedestal_macro prefix="${prefix}rob1_" tool="${tool}"/>
+        <xacro:za_pedestal_macro prefix="${prefix}rob2_" tool="${tool}"/>
+        <xacro:za_pedestal_macro prefix="${prefix}rob3_" tool="${tool}"/>
         <xacro:positioner_macro prefix="${prefix}"/>
+        <link name="${prefix}hydra_base"/>
+        <joint name="${prefix}hydra_base-rob1_pedestal_base" type="fixed">
+            <origin xyz="-${radius*sin(pi/6)} -${radius*cos(pi/6)}  0" rpy="0 0 ${pi/3}"/>
+            <parent link="${prefix}hydra_base"/>
+            <child  link="${prefix}rob1_pedestal_base"/>
+        </joint>
+        <joint name="${prefix}hydra_base-rob2_pedestal_base" type="fixed">
+            <origin xyz="${radius} 0 0" rpy="0 0 ${pi}"/>
+            <parent link="${prefix}hydra_base"/>
+            <child  link="${prefix}rob2_pedestal_base"/>
+        </joint>
+        <joint name="${prefix}hydra_base-rob3_pedestal_base" type="fixed">
+            <origin xyz="-${radius*sin(pi/6)} ${radius*cos(pi/6)} 0" rpy="0 0 -${pi/3}"/>
+            <parent link="${prefix}hydra_base"/>
+            <child  link="${prefix}rob3_pedestal_base"/>
+        </joint>
+        <joint name="${prefix}hydra_base-$(arg prefix)rotary_table_base" type="fixed">
+            <origin xyz="0 0 0"/>
+            <parent link="${prefix}hydra_base"/>
+            <child  link="${prefix}positioner_stand_base"/>
+        </joint>
     </xacro:macro>
 </robot>

Commit message: edit urdf to reflect ampf system

File: urdf/hydra.xacro (robot description, xacro)
@@ -2,5 +2,5 @@
 <robot name="hydra" xmlns:xacro="http://www.ros.org/wiki/xacro">
   <xacro:arg name="prefix" default=""/>
-  <xacro:property name="radius" value="0.95" />
+  <xacro:property name="radius" value="0.79375" />
   <xacro:property name="tool" default="typhoon_extruder" />
   <xacro:include filename="$(find hydra_description)/urdf/hydra_macro.xacro"/>

File: urdf/hydra_macro.xacro (robot description, xacro)
@@ -2,30 +2,41 @@
 <robot name="hydra" xmlns:xacro="http://www.ros.org/wiki/xacro">
     <xacro:include filename="$(find hydra_description)/urdf/robots/za_pedestal_macro.xacro"/>
-    <xacro:include filename="$(find hydra_description)/urdf/positioner/positioner_macro.xacro"/>
     <xacro:macro name="hydra_macro" params="prefix radius tool:='tool0'">
         <xacro:za_pedestal_macro prefix="${prefix}rob1_" tool="${tool}"/>
         <xacro:za_pedestal_macro prefix="${prefix}rob2_" tool="${tool}"/>
-        <xacro:za_pedestal_macro prefix="${prefix}rob3_" tool="${tool}"/>
-        <xacro:positioner_macro prefix="${prefix}"/>
         <link name="${prefix}hydra_base"/>
+        <link name="${prefix}optical_table"/>
+        <!-- link list -->
+        <link name="${prefix}optical_table_base">
+            <visual>
+                <geometry>
+                    <mesh filename="package://hydra_description/meshes/visual/optical_table.dae"/>
+                </geometry>
+            </visual>
+            <collision>
+                <geometry>
+                    <mesh filename="package://hydra_description/meshes/collision/optical_table.stl"/>
+                </geometry>
+            </collision>
+        </link>
+        <!-- joint list -->
+        <joint name="${prefix}hydra_base-optical_table_base" type="fixed">
+            <parent link="${prefix}hydra_base"/>
+            <child link="${prefix}optical_table_base"/>
+        </joint>
+        <joint name="${prefix}optical_table_base-optical_table" type="fixed">
+            <origin rpy="0.0 0.0 0.0" xyz="0 0 0.05842"/>
+            <parent link="${prefix}optical_table_base"/>
+            <child link="${prefix}optical_table"/>
+        </joint>
         <joint name="${prefix}hydra_base-rob1_pedestal_base" type="fixed">
-            <origin xyz="-${radius*sin(pi/6)} -${radius*cos(pi/6)}  0" rpy="0 0 ${pi/3}"/>
-            <parent link="${prefix}hydra_base"/>
+            <origin xyz="0 -${radius}  0" rpy="0 0 ${pi/2}"/>
+            <parent link="${prefix}optical_table"/>
             <child  link="${prefix}rob1_pedestal_base"/>
         </joint>
         <joint name="${prefix}hydra_base-rob2_pedestal_base" type="fixed">
-            <origin xyz="${radius} 0 0" rpy="0 0 ${pi}"/>
-            <parent link="${prefix}hydra_base"/>
+            <origin xyz="0 ${radius} 0" rpy="0 0 -${pi/2}"/>
+            <parent link="${prefix}optical_table"/>
             <child  link="${prefix}rob2_pedestal_base"/>
-        </joint>
-        <joint name="${prefix}hydra_base-rob3_pedestal_base" type="fixed">
-            <origin xyz="-${radius*sin(pi/6)} ${radius*cos(pi/6)} 0" rpy="0 0 -${pi/3}"/>
-            <parent link="${prefix}hydra_base"/>
-            <child  link="${prefix}rob3_pedestal_base"/>
-        </joint>
-        <joint name="${prefix}hydra_base-$(arg prefix)rotary_table_base" type="fixed">
-            <origin xyz="0 0 0"/>
-            <parent link="${prefix}hydra_base"/>
-            <child  link="${prefix}positioner_stand_base"/>
         </joint>
     </xacro:macro>

Commit message: add hydra_gazebo package

File: urdf/hydra.xacro (robot description, xacro)
@@ -11,3 +11,11 @@
       <child  link="$(arg prefix)hydra_base"/>
   </joint>
+  <!-- Gazebo plugin for ROS Control -->
+  <gazebo>
+    <plugin name="gazebo_ros_control" filename="libgazebo_ros_control.so">
+      <controlPeriod>0.001</controlPeriod>
+      <robotSimType>hydra_gazebo/HydraHWSim</robotSimType>
+    </plugin>
+    <self_collide>true</self_collide>
+  </gazebo>
 </robot>

File: urdf/positioner/positioner_macro.xacro (robot description, xacro)
@@ -2,4 +2,5 @@
 <robot xmlns:xacro="http://www.ros.org/wiki/xacro">
   <xacro:property name="pos_stand_height" value="0.32853" />
+  <xacro:include filename="$(find za_description)/urdf/utils.xacro"/>
   <xacro:macro name="positioner_macro" params="prefix">
     <!-- link list -->
@@ -15,4 +16,5 @@
           </geometry>
         </collision>
+        <xacro:default_inertial mass="1"/>
     </link>
     <link name="${prefix}rotary_table_base">
@@ -27,6 +29,9 @@
         </geometry>
       </collision>
+      <xacro:default_inertial mass="1"/>
     </link>
-    <link name="${prefix}rotary_table_top"/>
+    <link name="${prefix}rotary_table_top">
+      <xacro:default_inertial mass="1"/>
+    </link>
     <link name="${prefix}positioner_base">
         <visual>
@@ -40,4 +45,9 @@
         </geometry>
       </collision>
+      <inertial>
+        <origin xyz="0.000000 0.000000 0.006349"/>
+        <mass value="27.67"/>
+        <inertia ixx="1.929232" ixy="0.000000" ixz="0.000000" iyy="1.929232" iyz="0.000000" izz="3.857721"/>
+      </inertial>
     </link>
     <link name="${prefix}positioner"/>
@@ -71,4 +81,5 @@
       <child link="${prefix}positioner_static"/>
     </joint>
+    <xacro:gazebo-joint joint="${prefix}rotary_table_positioner" transmission="hardware_interface/VelocityJointInterface"/>
   </xacro:macro>
 </robot>

File: urdf/robots/za_tool.xacro (robot description, xacro)
@@ -5,3 +5,19 @@
   <xacro:include filename="$(find hydra_description)/urdf/robots/za_tool_macro.xacro" />
   <xacro:za_tool_macro prefix="$(arg prefix)" tool="$(arg tool)"/>
+  <!-- 'world' frame: default pose reference frame -->
+  <link name="world" />
+  <joint name="world-$(arg prefix)base_link" type="fixed">
+    <origin xyz="0 0 0" rpy="0 0 0"/>
+    <axis xyz="0 0 1"/>
+    <parent link="world"/>
+    <child link="$(arg prefix)base_link"/>
+  </joint>
+  <!-- Gazebo plugin for ROS Control -->
+  <gazebo>
+    <plugin name="gazebo_ros_control" filename="libgazebo_ros_control.so">
+      <controlPeriod>0.001</controlPeriod>
+      <robotSimType>za_gazebo/ZaHWSim</robotSimType>
+    </plugin>
+    <self_collide>true</self_collide>
+  </gazebo>
 </robot>

File: urdf/tools/typhoon_extruder_macro.xacro (robot description, xacro)
@@ -5,5 +5,5 @@
 	<xacro:macro name="typhoon_extruder_macro" params="prefix">
 		<!-- link list -->
-		<link name="${prefix}typhoon_extruder_base">
+		<link name="${prefix}typhoon_extruder">
 			<visual>
 				<geometry>
@@ -16,16 +16,21 @@
 				</geometry>
 			</collision>
+			<inertial>
+    			<origin xyz="0.065346 0.000016 -0.031645"/>
+    			<mass value="1.75"/>
+				<inertia ixx="0.006265" ixy="0.000003" ixz="-0.000805" iyy="0.006649" iyz="0.000002" izz="0.001704"/>
+			</inertial>
 		</link>
-		<link name="${prefix}typhoon_extruder" />
+		<link name="${prefix}typhoon_extruder_tcp" />
 		<!-- attach extruder to flange -->
 		<joint name="${prefix}extruder_attach_joint" type="fixed">
 			<origin xyz="0 0 0" rpy="0 0 0" />
 			<parent link="${prefix}flange"/>
-			<child link="${prefix}typhoon_extruder_base"/>
+			<child link="${prefix}typhoon_extruder"/>
 		</joint>
 		<joint name="${prefix}extruder_extruder_base" type="fixed">
 			<origin xyz="${tcp_trans}" rpy="${tcp_rot}" />
-			<parent link="${prefix}typhoon_extruder_base"/>
-			<child link="${prefix}typhoon_extruder"/>
+			<parent link="${prefix}typhoon_extruder"/>
+			<child link="${prefix}typhoon_extruder_tcp"/>
 		</joint>
 	</xacro:macro>

Commit message: change default tool to flange

File: urdf/hydra.xacro (robot description, xacro)
@@ -3,5 +3,5 @@
   <xacro:arg name="prefix" default=""/>
   <xacro:property name="radius" value="0.79375" />
-  <xacro:property name="tool" default="typhoon_extruder" />
+  <xacro:property name="tool" default="flange" />
   <xacro:include filename="$(find hydra_description)/urdf/hydra_macro.xacro"/>
   <xacro:hydra_macro prefix="$(arg prefix)" radius="${radius}" tool="${tool}"/>
