Commit message: remove optical table and add h-frame bases

File: urdf/hydra.xacro (robot description, xacro)
@@ -2,6 +2,6 @@
 <robot name="hydra" xmlns:xacro="http://www.ros.org/wiki/xacro">
   <xacro:arg name="prefix" default=""/>
-  <xacro:property name="radius" value="0.79375" />
-  <xacro:property name="tool" default="flange" />
+  <xacro:property name="radius" value="0.825"/>
+  <xacro:property name="tool" default="typhoon_extruder" />
   <xacro:include filename="$(find hydra_description)/urdf/hydra_macro.xacro"/>
   <xacro:hydra_macro prefix="$(arg prefix)" radius="${radius}" tool="${tool}"/>
@@ -10,4 +10,10 @@
       <parent link="world"/>
       <child  link="$(arg prefix)hydra_base"/>
+  </joint>
+  <link name="work_object"/>
+  <joint name="world-$(arg prefix)work_object" type="fixed">
+    <origin xyz="0 0 0.9" rpy="0 0 0"/>
+    <parent link="world"/>
+    <child  link="$(arg prefix)work_object"/>
   </joint>
   <!-- Gazebo plugin for ROS Control -->

File: urdf/hydra_macro.xacro (robot description, xacro)
@@ -8,36 +8,13 @@
         <xacro:za_pedestal_macro prefix="${prefix}rob2_" tool="${tool}"/>
         <link name="${prefix}hydra_base"/>
-        <link name="${prefix}optical_table"/>
-        <!-- link list -->
-        <link name="${prefix}optical_table_base">
-            <visual>
-                <geometry>
-                    <mesh filename="package://hydra_description/meshes/visual/optical_table.dae"/>
-                </geometry>
-            </visual>
-            <collision>
-                <geometry>
-                    <mesh filename="package://hydra_description/meshes/collision/optical_table.stl"/>
-                </geometry>
-            </collision>
-        </link>
         <!-- joint list -->
-        <joint name="${prefix}hydra_base-optical_table_base" type="fixed">
-            <parent link="${prefix}hydra_base"/>
-            <child link="${prefix}optical_table_base"/>
-        </joint>
-        <joint name="${prefix}optical_table_base-optical_table" type="fixed">
-            <origin rpy="0.0 0.0 0.0" xyz="0 0 0.05842"/>
-            <parent link="${prefix}optical_table_base"/>
-            <child link="${prefix}optical_table"/>
-        </joint>
         <joint name="${prefix}hydra_base-rob1_pedestal_base" type="fixed">
             <origin xyz="0 -${radius}  0" rpy="0 0 ${pi/2}"/>
-            <parent link="${prefix}optical_table"/>
+            <parent link="${prefix}hydra_base"/>
             <child  link="${prefix}rob1_pedestal_base"/>
         </joint>
         <joint name="${prefix}hydra_base-rob2_pedestal_base" type="fixed">
             <origin xyz="0 ${radius} 0" rpy="0 0 -${pi/2}"/>
-            <parent link="${prefix}optical_table"/>
+            <parent link="${prefix}hydra_base"/>
             <child  link="${prefix}rob2_pedestal_base"/>
         </joint>

File: urdf/robots/za_pedestal_macro.xacro (robot description, xacro)
@@ -1,30 +1,48 @@
 <?xml version="1.0"?>
 <robot xmlns:xacro="http://www.ros.org/wiki/xacro">
-    <xacro:property name="ped_height" value="0.585" />
+  <xacro:property name="ped_height" value="0.585"/>
+  <xacro:property name="base_height" value="0.2"/>
 	<xacro:macro name="za_pedestal_macro" params="prefix tool:='tool0'" >
 		<xacro:include filename="$(find hydra_description)/urdf/robots/za_tool_macro.xacro" />
 		<xacro:za_tool_macro prefix="${prefix}" tool="${tool}"/>
-        <link name="${prefix}pedestal_base">
-            <visual>
-                <geometry>
-                    <mesh filename="package://hydra_description/meshes/visual/za_pedestal.dae"/>
-                </geometry>
-            </visual>
-            <collision>
-                <geometry>
-                    <mesh filename="package://hydra_description/meshes/collision/za_pedestal_collision.stl"/>
-                </geometry>
-            </collision>
-        </link>
+    <link name="${prefix}pedestal_base">
+      <visual>
+        <geometry>
+          <mesh filename="package://hydra_description/meshes/visual/hframe_base.dae"/>
+        </geometry>
+      </visual>
+      <collision>
+        <geometry>
+          <mesh filename="package://hydra_description/meshes/collision/optical_table.stl"/>
+        </geometry>
+      </collision>
+    </link>
+    <link name="${prefix}pedestal">
+      <visual>
+        <geometry>
+          <mesh filename="package://hydra_description/meshes/visual/za_pedestal.dae"/>
+        </geometry>
+      </visual>
+      <collision>
+        <geometry>
+          <mesh filename="package://hydra_description/meshes/collision/za_pedestal_collision.stl"/>
+        </geometry>
+      </collision>
+    </link>
 		<link name="${prefix}pedestal_top"/>
-        <joint name="${prefix}pedestal_base-${prefix}pedestal_top" type="fixed">
-            <origin rpy="0.0 0.0 0.0" xyz="0 0 ${ped_height}"/>
-            <parent link="${prefix}pedestal_base"/>
-            <child  link="${prefix}pedestal_top"/>
-        </joint>
-        <joint name="${prefix}pedestal_top-${prefix}base_link" type="fixed">
-            <parent link="${prefix}pedestal_top"/>
-            <child  link="${prefix}base_link"/>
-        </joint>
+    <joint name="${prefix}pedestal_base-${prefix}pedestal" type="fixed">
+      <origin rpy="0.0 0.0 0.0" xyz="0 0 ${base_height}"/>
+      <parent link="${prefix}pedestal_base"/>
+      <child  link="${prefix}pedestal"/>
+    </joint>
+    <joint name="${prefix}pedestal-${prefix}pedestal_top" type="fixed">
+      <origin rpy="0.0 0.0 0.0" xyz="0 0 ${ped_height}"/>
+      <parent link="${prefix}pedestal"/>
+      <child  link="${prefix}pedestal_top"/>
+    </joint>
+    <joint name="${prefix}pedestal_top-${prefix}base_link" type="fixed">
+      <parent link="${prefix}pedestal_top"/>
+      <child  link="${prefix}base_link"/>
+    </joint>
 	</xacro:macro>
 </robot>

Commit message: change robot spacing

File: urdf/hydra.xacro (robot description, xacro)
@@ -2,5 +2,5 @@
 <robot name="hydra" xmlns:xacro="http://www.ros.org/wiki/xacro">
   <xacro:arg name="prefix" default=""/>
-  <xacro:property name="radius" value="0.825"/>
+  <xacro:property name="radius" value="0.75"/>
   <xacro:property name="tool" default="typhoon_extruder" />
   <xacro:include filename="$(find hydra_description)/urdf/hydra_macro.xacro"/>
@@ -13,5 +13,5 @@
   <link name="work_object"/>
   <joint name="world-$(arg prefix)work_object" type="fixed">
-    <origin xyz="0 0 0.9" rpy="0 0 0"/>
+    <origin xyz="0 0 0.8" rpy="0 0 0"/>
     <parent link="world"/>
     <child  link="$(arg prefix)work_object"/>

Commit message: third robot holds the positioner table

File: urdf/hydra.xacro (robot description, xacro)
@@ -2,5 +2,5 @@
 <robot name="hydra" xmlns:xacro="http://www.ros.org/wiki/xacro">
   <xacro:arg name="prefix" default=""/>
-  <xacro:property name="radius" value="0.95" />
+  <xacro:property name="radius" value="0.85" />
   <xacro:property name="tool" default="typhoon_extruder" />
   <xacro:include filename="$(find hydra_description)/urdf/hydra_macro.xacro"/>

File: urdf/hydra_macro.xacro (robot description, xacro)
@@ -2,45 +2,39 @@
 <robot name="hydra" xmlns:xacro="http://www.ros.org/wiki/xacro">
     <xacro:include filename="$(find hydra_description)/urdf/robots/za_pedestal_macro.xacro"/>
-    <xacro:include filename="$(find hydra_description)/urdf/positioner/positioner_macro.xacro"/>
+    <xacro:include filename="$(find hydra_description)/urdf/robots/za_positioner_macro.xacro"/>
     <xacro:macro name="hydra_macro" params="prefix radius tool:='tool0'">
-        <!-- Is the robot being simulated in gazebo? -->
-        <xacro:arg name="gazebo" default="true" />
-        <xacro:za_pedestal_macro prefix="${prefix}rob1_" tool="${tool}"/>
-        <xacro:za_pedestal_macro prefix="${prefix}rob2_" tool="${tool}"/>
-        <xacro:za_pedestal_macro prefix="${prefix}rob3_" tool="${tool}"/>
-        <xacro:positioner_macro prefix="${prefix}"/>
-        <link name="${prefix}hydra_base"/>
-        <joint name="${prefix}hydra_base-rob1_pedestal_base" type="fixed">
-            <origin xyz="-${radius*sin(pi/6)} -${radius*cos(pi/6)}  0" rpy="0 0 ${pi/3}"/>
-            <parent link="${prefix}hydra_base"/>
-            <child  link="${prefix}rob1_pedestal_base"/>
-        </joint>
-        <joint name="${prefix}hydra_base-rob2_pedestal_base" type="fixed">
-            <origin xyz="${radius} 0 0" rpy="0 0 ${pi}"/>
-            <parent link="${prefix}hydra_base"/>
-            <child  link="${prefix}rob2_pedestal_base"/>
-        </joint>
-        <joint name="${prefix}hydra_base-rob3_pedestal_base" type="fixed">
-            <origin xyz="-${radius*sin(pi/6)} ${radius*cos(pi/6)} 0" rpy="0 0 -${pi/3}"/>
-            <parent link="${prefix}hydra_base"/>
-            <child  link="${prefix}rob3_pedestal_base"/>
-        </joint>
-        <joint name="${prefix}hydra_base-$(arg prefix)rotary_table_base" type="fixed">
-            <origin xyz="0 0 0"/>
-            <parent link="${prefix}hydra_base"/>
-            <child  link="${prefix}positioner_stand_base"/>
-        </joint>
-        <xacro:if value="$(arg gazebo)">
-            <transmission name="${prefix}hydra_model">
-              <type>hydra_hw/HydraModelInterface</type>
-              <joint name="${prefix}positioner_joint">
-                <role>positioner</role>
-                <hardwareInterface>hydra_hw/HydraModelInterface</hardwareInterface>
-              </joint>
-              <actuator name="${prefix}_motor_positioner_joint">
-                <hardwareInterface>hydra_hw/HydraModelInterface</hardwareInterface>
-              </actuator>
-            </transmission>
-        </xacro:if>
+      <!-- Is the robot being simulated in gazebo? -->
+      <xacro:arg name="gazebo" default="true" />
+      <xacro:za_pedestal_macro prefix="${prefix}rob1_" tool="${tool}"/>
+      <xacro:za_pedestal_macro prefix="${prefix}rob2_" tool="${tool}"/>
+      <xacro:za_positioner_macro prefix="${prefix}rob3_"/>
+      <link name="${prefix}hydra_base"/>
+      <joint name="${prefix}hydra_base-rob1_pedestal_base" type="fixed">
+        <origin xyz="0 -${radius} 0.1" rpy="0 0 ${pi/2}"/>
+        <parent link="${prefix}hydra_base"/>
+        <child  link="${prefix}rob1_pedestal_base"/>
+      </joint>
+      <joint name="${prefix}hydra_base-rob2_pedestal_base" type="fixed">
+        <origin xyz="0 ${radius} 0.1" rpy="0 0 -${pi/2}"/>
+        <parent link="${prefix}hydra_base"/>
+        <child  link="${prefix}rob2_pedestal_base"/>
+      </joint>
+      <joint name="${prefix}hydra_base-rob3_base_link" type="fixed">
+        <origin xyz="0 0 0" rpy="0 0 0"/>
+        <parent link="${prefix}hydra_base"/>
+        <child  link="${prefix}rob3_base_link"/>
+      </joint>
+      <xacro:if value="$(arg gazebo)">
+        <transmission name="${prefix}hydra_model">
+          <type>hydra_hw/HydraModelInterface</type>
+          <joint name="${prefix}positioner_joint">
+            <role>positioner</role>
+            <hardwareInterface>hydra_hw/HydraModelInterface</hardwareInterface>
+          </joint>
+          <actuator name="${prefix}_motor_positioner_joint">
+            <hardwareInterface>hydra_hw/HydraModelInterface</hardwareInterface>
+          </actuator>
+        </transmission>
+      </xacro:if>
     </xacro:macro>
-</robot>
+  </robot>
