Commit message: port to ros2

File: urdf/hydra.xacro (robot description, xacro)
@@ -4,18 +4,18 @@
   <xacro:property name="radius" value="0.95" />
   <xacro:property name="tool" default="typhoon_extruder" />
+  <!-- ros2_control parameters-->
+  <xacro:arg name="use_mock_hardware" default="true"/>
+  <xacro:arg name="include_hardware" default="true"/>
   <xacro:include filename="$(find hydra_description)/urdf/hydra_macro.xacro"/>
-  <xacro:hydra_macro prefix="$(arg prefix)" radius="${radius}" tool="${tool}"/>
+  <xacro:hydra_macro prefix="$(arg prefix)"
+    radius="${radius}"
+    tool="${tool}"
+    include_hardware="$(arg include_hardware)"
+    use_mock_hardware="$(arg use_mock_hardware)"
+  />
   <link name="world"/>
   <joint name="world-$(arg prefix)hydra_base" type="fixed">
-      <parent link="world"/>
-      <child  link="$(arg prefix)hydra_base"/>
+    <parent link="world"/>
+    <child  link="$(arg prefix)hydra_base"/>
   </joint>
-  <!-- Gazebo plugin for ROS Control -->
-  <gazebo>
-    <plugin name="gazebo_ros_control" filename="libgazebo_ros_control.so">
-      <controlPeriod>0.001</controlPeriod>
-      <robotSimType>hydra_gazebo/HydraHWSim</robotSimType>
-    </plugin>
-    <self_collide>true</self_collide>
-  </gazebo>
 </robot>

File: urdf/hydra_macro.xacro (robot description, xacro)
@@ -1,46 +1,45 @@
 <?xml version="1.0" ?>
 <robot name="hydra" xmlns:xacro="http://www.ros.org/wiki/xacro">
-    <xacro:include filename="$(find hydra_description)/urdf/robots/za_pedestal_macro.xacro"/>
-    <xacro:include filename="$(find hydra_description)/urdf/positioner/positioner_macro.xacro"/>
-    <xacro:macro name="hydra_macro" params="prefix radius tool:='tool0'">
-        <!-- Is the robot being simulated in gazebo? -->
-        <xacro:arg name="gazebo" default="true" />
-        <xacro:za_pedestal_macro prefix="${prefix}rob1_" tool="${tool}"/>
-        <xacro:za_pedestal_macro prefix="${prefix}rob2_" tool="${tool}"/>
-        <xacro:za_pedestal_macro prefix="${prefix}rob3_" tool="${tool}"/>
-        <xacro:positioner_macro prefix="${prefix}"/>
-        <link name="${prefix}hydra_base"/>
-        <joint name="${prefix}hydra_base-rob1_pedestal_base" type="fixed">
-            <origin xyz="-${radius*sin(pi/6)} -${radius*cos(pi/6)}  0" rpy="0 0 ${pi/3}"/>
-            <parent link="${prefix}hydra_base"/>
-            <child  link="${prefix}rob1_pedestal_base"/>
-        </joint>
-        <joint name="${prefix}hydra_base-rob2_pedestal_base" type="fixed">
-            <origin xyz="${radius} 0 0" rpy="0 0 ${pi}"/>
-            <parent link="${prefix}hydra_base"/>
-            <child  link="${prefix}rob2_pedestal_base"/>
-        </joint>
-        <joint name="${prefix}hydra_base-rob3_pedestal_base" type="fixed">
-            <origin xyz="-${radius*sin(pi/6)} ${radius*cos(pi/6)} 0" rpy="0 0 -${pi/3}"/>
-            <parent link="${prefix}hydra_base"/>
-            <child  link="${prefix}rob3_pedestal_base"/>
-        </joint>
-        <joint name="${prefix}hydra_base-$(arg prefix)rotary_table_base" type="fixed">
-            <origin xyz="0 0 0"/>
-            <parent link="${prefix}hydra_base"/>
-            <child  link="${prefix}positioner_stand_base"/>
-        </joint>
-        <xacro:if value="$(arg gazebo)">
-            <transmission name="${prefix}hydra_model">
-              <type>hydra_hw/HydraModelInterface</type>
-              <joint name="${prefix}positioner_joint">
-                <role>positioner</role>
-                <hardwareInterface>hydra_hw/HydraModelInterface</hardwareInterface>
-              </joint>
-              <actuator name="${prefix}_motor_positioner_joint">
-                <hardwareInterface>hydra_hw/HydraModelInterface</hardwareInterface>
-              </actuator>
-            </transmission>
-        </xacro:if>
-    </xacro:macro>
+  <xacro:include filename="$(find hydra_description)/urdf/robots/za_pedestal_macro.xacro"/>
+  <xacro:include filename="$(find hydra_description)/urdf/positioner/positioner_macro.xacro"/>
+  <xacro:macro name="hydra_macro" params="
+    prefix
+    radius
+    tool:='tool0'
+    include_hardware:=false
+    use_mock_hardware:=true">
+    <xacro:za_pedestal_macro prefix="${prefix}rob1_" tool="${tool}"/>
+    <xacro:za_pedestal_macro prefix="${prefix}rob2_" tool="${tool}"/>
+    <xacro:za_pedestal_macro prefix="${prefix}rob3_" tool="${tool}"/>
+    <xacro:positioner_macro prefix="${prefix}"/>
+    <link name="${prefix}hydra_base"/>
+    <joint name="${prefix}hydra_base-rob1_pedestal_base" type="fixed">
+      <origin xyz="-${radius*sin(pi/6)} -${radius*cos(pi/6)}  0" rpy="0 0 ${pi/3}"/>
+      <parent link="${prefix}hydra_base"/>
+      <child  link="${prefix}rob1_pedestal_base"/>
+    </joint>
+    <joint name="${prefix}hydra_base-rob2_pedestal_base" type="fixed">
+      <origin xyz="${radius} 0 0" rpy="0 0 ${pi}"/>
+      <parent link="${prefix}hydra_base"/>
+      <child  link="${prefix}rob2_pedestal_base"/>
+    </joint>
+    <joint name="${prefix}hydra_base-rob3_pedestal_base" type="fixed">
+      <origin xyz="-${radius*sin(pi/6)} ${radius*cos(pi/6)} 0" rpy="0 0 -${pi/3}"/>
+      <parent link="${prefix}hydra_base"/>
+      <child  link="${prefix}rob3_pedestal_base"/>
+    </joint>
+    <joint name="${prefix}hydra_base-$(arg prefix)rotary_table_base" type="fixed">
+      <origin xyz="0 0 0"/>
+      <parent link="${prefix}hydra_base"/>
+      <child  link="${prefix}positioner_stand_base"/>
+    </joint>
+    <xacro:if value="${include_hardware}">
+      <xacro:include filename="$(find za_description)/urdf/za.ros2_control.xacro"/>
+      <xacro:za_ros2_control prefix="${prefix}rob1_" use_mock_hardware="${use_mock_hardware}"/>
+      <xacro:za_ros2_control prefix="${prefix}rob2_" use_mock_hardware="${use_mock_hardware}"/>
+      <xacro:za_ros2_control prefix="${prefix}rob3_" use_mock_hardware="${use_mock_hardware}"/>
+      <xacro:include filename="$(find hydra_description)/urdf/positioner/positioner.ros2_control.xacro"/>
+      <xacro:positioner_ros2_control prefix="${prefix}" use_mock_hardware="${use_mock_hardware}"/>
+    </xacro:if>
+  </xacro:macro>
 </robot>

File: urdf/positioner/positioner.xacro (robot description, xacro)
@@ -2,4 +2,7 @@
 <robot name="hydra_positioner" xmlns:xacro="http://www.ros.org/wiki/xacro">
   <xacro:arg name="prefix" default=""/>
+  <!-- ros2_control parameters-->
+  <xacro:arg name="use_mock_hardware" default="true"/>
+  <xacro:arg name="include_hardware" default="true"/>
   <xacro:include filename="$(find hydra_description)/urdf/positioner/positioner_macro.xacro"/>
   <xacro:positioner_macro prefix="$(arg prefix)"/>
@@ -9,3 +12,7 @@
     <child link="$(arg prefix)positioner_stand_base"/>
   </joint>
+  <xacro:if value="$(arg include_hardware)">
+    <xacro:include filename="$(find hydra_description)/urdf/positioner/positioner.ros2_control.xacro"/>
+    <xacro:positioner_ros2_control prefix="$(arg prefix)" use_mock_hardware="$(arg use_mock_hardware)"/>
+  </xacro:if>
 </robot>

File: urdf/positioner/positioner_macro.xacro (robot description, xacro)
@@ -4,22 +4,20 @@
   <xacro:include filename="$(find za_description)/urdf/utils.xacro"/>
   <xacro:macro name="positioner_macro" params="prefix">
-    <!-- Is the robot being simulated in gazebo?" -->
-    <xacro:arg name="gazebo" default="true" />
     <!-- link list -->
     <link name="${prefix}positioner_stand_base">
-        <visual>
-          <geometry>
-            <mesh filename="package://hydra_description/meshes/visual/positioner_stand.dae"/>
-          </geometry>
-        </visual>
-        <collision>
-          <geometry>
-            <mesh filename="package://hydra_description/meshes/collision/positioner_stand_collision.stl"/>
-          </geometry>
-        </collision>
-        <xacro:default_inertial mass="1"/>
+      <visual>
+        <geometry>
+          <mesh filename="package://hydra_description/meshes/visual/positioner_stand.dae"/>
+        </geometry>
+      </visual>
+      <collision>
+        <geometry>
+          <mesh filename="package://hydra_description/meshes/collision/positioner_stand_collision.stl"/>
+        </geometry>
+      </collision>
+      <xacro:default_inertial mass="1"/>
     </link>
     <link name="${prefix}rotary_table_base">
-        <visual>
+      <visual>
         <geometry>
           <mesh filename="package://hydra_description/meshes/visual/rotary_table.dae"/>
@@ -37,5 +35,5 @@
     </link>
     <link name="${prefix}positioner_base">
-        <visual>
+      <visual>
         <geometry>
           <mesh filename="package://hydra_description/meshes/visual/hydra_positioner.dae"/>
@@ -67,5 +65,4 @@
     </joint>
     <joint name="${prefix}positioner_joint" type="continuous">
-    <!--<joint name="${prefix}rotary_table_positioner" type="continuous">-->
       <origin rpy="0.0 0.0 0.0" xyz="0 0 0"/>
       <axis xyz="0 0 1"/>
@@ -84,15 +81,4 @@
       <child link="${prefix}positioner_static"/>
     </joint>
-    <!-- Define additional Gazebo tags -->
-    <xacro:if value="$(arg gazebo)">
-      <xacro:gazebo-joint joint="${prefix}positioner_joint" transmission="hardware_interface/EffortJointInterface"/>
-      <xacro:gazebo-joint joint="${prefix}positioner_joint" transmission="hardware_interface/VelocityJointInterface"/>
-      <xacro:gazebo-joint joint="${prefix}positioner_joint" transmission="hardware_interface/PositionJointInterface"/>
-      <transmission name="${prefix}positioner_state">
-        <type>hydra_hw/PositionerStateInterface</type>
-        <joint name="${prefix}positioner_joint"><hardwareInterface>hydra_hw/PositionerStateInterface</hardwareInterface></joint>
-        <actuator name="${prefix}positioner_motor"><hardwareInterface>hydra_hw/PositionerStateInterface</hardwareInterface></actuator>
-      </transmission>
-    </xacro:if>
   </xacro:macro>
 </robot>

File: urdf/robots/za_pedestal.xacro (robot description, xacro)
@@ -3,5 +3,12 @@
   <xacro:arg name="prefix" default="" />
   <xacro:arg name="tool" default="typhoon_extruder" />
+  <!-- ros2_control parameters-->
+  <xacro:arg name="use_mock_hardware" default="true"/>
+  <xacro:arg name="include_hardware" default="true"/>
   <xacro:include filename="$(find hydra_description)/urdf/robots/za_pedestal_macro.xacro" />
   <xacro:za_pedestal_macro prefix="$(arg prefix)" tool="$(arg tool)"/>
+  <xacro:if value="$(arg include_hardware)">
+    <xacro:include filename="$(find za_description)/urdf/za.ros2_control.xacro"/>
+    <xacro:za_ros2_control prefix="$(arg prefix)" use_mock_hardware="$(arg use_mock_hardware)"/>
+  </xacro:if>
 </robot>

File: urdf/robots/za_pedestal_macro.xacro (robot description, xacro)
@@ -1,30 +1,30 @@
 <?xml version="1.0"?>
 <robot xmlns:xacro="http://www.ros.org/wiki/xacro">
-    <xacro:property name="ped_height" value="0.585" />
+  <xacro:property name="ped_height" value="0.585" />
 	<xacro:macro name="za_pedestal_macro" params="prefix tool:='tool0'" >
 		<xacro:include filename="$(find hydra_description)/urdf/robots/za_tool_macro.xacro" />
 		<xacro:za_tool_macro prefix="${prefix}" tool="${tool}"/>
-        <link name="${prefix}pedestal_base">
-            <visual>
-                <geometry>
-                    <mesh filename="package://hydra_description/meshes/visual/za_pedestal.dae"/>
-                </geometry>
-            </visual>
-            <collision>
-                <geometry>
-                    <mesh filename="package://hydra_description/meshes/collision/za_pedestal_collision.stl"/>
-                </geometry>
-            </collision>
-        </link>
+    <link name="${prefix}pedestal_base">
+      <visual>
+        <geometry>
+          <mesh filename="package://hydra_description/meshes/visual/za_pedestal.dae"/>
+        </geometry>
+      </visual>
+      <collision>
+        <geometry>
+          <mesh filename="package://hydra_description/meshes/collision/za_pedestal_collision.stl"/>
+        </geometry>
+      </collision>
+    </link>
 		<link name="${prefix}pedestal_top"/>
-        <joint name="${prefix}pedestal_base-${prefix}pedestal_top" type="fixed">
-            <origin rpy="0.0 0.0 0.0" xyz="0 0 ${ped_height}"/>
-            <parent link="${prefix}pedestal_base"/>
-            <child  link="${prefix}pedestal_top"/>
-        </joint>
-        <joint name="${prefix}pedestal_top-${prefix}base_link" type="fixed">
-            <parent link="${prefix}pedestal_top"/>
-            <child  link="${prefix}base_link"/>
-        </joint>
+    <joint name="${prefix}pedestal_base-${prefix}pedestal_top" type="fixed">
+      <origin rpy="0.0 0.0 0.0" xyz="0 0 ${ped_height}"/>
+      <parent link="${prefix}pedestal_base"/>
+      <child  link="${prefix}pedestal_top"/>
+    </joint>
+    <joint name="${prefix}pedestal_top-${prefix}base_link" type="fixed">
+      <parent link="${prefix}pedestal_top"/>
+      <child  link="${prefix}base_link"/>
+    </joint>
 	</xacro:macro>
 </robot>

File: urdf/robots/za_tool_macro.xacro (robot description, xacro)
@@ -3,5 +3,5 @@
 	<xacro:macro name="za_tool_macro" params="prefix tool:='tool0'" >
 		<xacro:include filename="$(find za_description)/urdf/za_macro.xacro" />
-		<xacro:za_macro prefix="${prefix}" />
+		<xacro:za_macro prefix="${prefix}"/>
 		<xml:property name="var" value="typhoon_extruder"/>
 		<xacro:if value="${tool == 'typhoon_extruder'}">
@@ -9,4 +9,4 @@
 			<xacro:typhoon_extruder_macro prefix="${prefix}" />
 		</xacro:if>
-	</xacro:macro>
+  </xacro:macro>
 </robot>

Commit message: port to ros2

File: urdf/hydra.xacro (robot description, xacro)
@@ -2,12 +2,20 @@
 <robot name="hydra" xmlns:xacro="http://www.ros.org/wiki/xacro">
   <xacro:arg name="prefix" default=""/>
-  <xacro:property name="radius" value="0.75"/>
+  <xacro:property name="radius" value="0.75" />
   <xacro:property name="tool" default="typhoon_extruder" />
+  <!-- ros2_control parameters-->
+  <xacro:arg name="use_mock_hardware" default="true"/>
+  <xacro:arg name="include_hardware" default="true"/>
   <xacro:include filename="$(find hydra_description)/urdf/hydra_macro.xacro"/>
-  <xacro:hydra_macro prefix="$(arg prefix)" radius="${radius}" tool="${tool}"/>
+  <xacro:hydra_macro prefix="$(arg prefix)"
+    radius="${radius}"
+    tool="${tool}"
+    include_hardware="$(arg include_hardware)"
+    use_mock_hardware="$(arg use_mock_hardware)"
+  />
   <link name="world"/>
   <joint name="world-$(arg prefix)hydra_base" type="fixed">
-      <parent link="world"/>
-      <child  link="$(arg prefix)hydra_base"/>
+    <parent link="world"/>
+    <child  link="$(arg prefix)hydra_base"/>
   </joint>
   <link name="work_object"/>
@@ -17,11 +25,3 @@
     <child  link="$(arg prefix)work_object"/>
   </joint>
-  <!-- Gazebo plugin for ROS Control -->
-  <gazebo>
-    <plugin name="gazebo_ros_control" filename="libgazebo_ros_control.so">
-      <controlPeriod>0.001</controlPeriod>
-      <robotSimType>hydra_gazebo/HydraHWSim</robotSimType>
-    </plugin>
-    <self_collide>true</self_collide>
-  </gazebo>
 </robot>

File: urdf/hydra_macro.xacro (robot description, xacro)
@@ -1,34 +1,29 @@
 <?xml version="1.0" ?>
 <robot name="hydra" xmlns:xacro="http://www.ros.org/wiki/xacro">
-    <xacro:include filename="$(find hydra_description)/urdf/robots/za_pedestal_macro.xacro"/>
-    <xacro:macro name="hydra_macro" params="prefix radius tool:='tool0'">
-        <!-- Is the robot being simulated in gazebo? -->
-        <xacro:arg name="gazebo" default="true" />
-        <xacro:za_pedestal_macro prefix="${prefix}rob1_" tool="${tool}"/>
-        <xacro:za_pedestal_macro prefix="${prefix}rob2_" tool="${tool}"/>
-        <link name="${prefix}hydra_base"/>
-        <!-- joint list -->
-        <joint name="${prefix}hydra_base-rob1_pedestal_base" type="fixed">
-            <origin xyz="0 -${radius}  0" rpy="0 0 ${pi/2}"/>
-            <parent link="${prefix}hydra_base"/>
-            <child  link="${prefix}rob1_pedestal_base"/>
-        </joint>
-        <joint name="${prefix}hydra_base-rob2_pedestal_base" type="fixed">
-            <origin xyz="0 ${radius} 0" rpy="0 0 -${pi/2}"/>
-            <parent link="${prefix}hydra_base"/>
-            <child  link="${prefix}rob2_pedestal_base"/>
-        </joint>
-        <xacro:if value="$(arg gazebo)">
-            <transmission name="${prefix}hydra_model">
-              <type>hydra_hw/HydraModelInterface</type>
-              <joint name="${prefix}positioner_joint">
-                <role>positioner</role>
-                <hardwareInterface>hydra_hw/HydraModelInterface</hardwareInterface>
-              </joint>
-              <actuator name="${prefix}_motor_positioner_joint">
-                <hardwareInterface>hydra_hw/HydraModelInterface</hardwareInterface>
-              </actuator>
-            </transmission>
-        </xacro:if>
-    </xacro:macro>
+  <xacro:include filename="$(find hydra_description)/urdf/robots/za_pedestal_macro.xacro"/>
+  <xacro:macro name="hydra_macro" params="
+    prefix
+    radius
+    tool:='tool0'
+    include_hardware:=false
+    use_mock_hardware:=true">
+    <xacro:za_pedestal_macro prefix="${prefix}rob1_" tool="${tool}"/>
+    <xacro:za_pedestal_macro prefix="${prefix}rob2_" tool="${tool}"/>
+    <link name="${prefix}hydra_base"/>
+    <joint name="${prefix}hydra_base-rob1_pedestal_base" type="fixed">
+      <origin xyz="0 -${radius}  0" rpy="0 0 ${pi/2}"/>
+      <parent link="${prefix}world"/>
+      <child  link="${prefix}rob1_pedestal_base"/>
+    </joint>
+    <joint name="${prefix}hydra_base-rob2_pedestal_base" type="fixed">
+      <origin xyz="0 ${radius} 0" rpy="0 0 -${pi/2}"/>
+      <parent link="${prefix}world"/>
+      <child  link="${prefix}rob2_pedestal_base"/>
+    </joint>
+    <xacro:if value="${include_hardware}">
+      <xacro:include filename="$(find za_description)/urdf/za.ros2_control.xacro"/>
+      <xacro:za_ros2_control prefix="${prefix}rob1_" use_mock_hardware="${use_mock_hardware}"/>
+      <xacro:za_ros2_control prefix="${prefix}rob2_" use_mock_hardware="${use_mock_hardware}"/>
+    </xacro:if>
+  </xacro:macro>
 </robot>

File: urdf/robots/za_tool.xacro (robot description, xacro)
@@ -3,5 +3,8 @@
   <xacro:arg name="prefix" default="" />
   <xacro:arg name="tool" default="typhoon_extruder" />
-  <xacro:include filename="$(find hydra_description)/urdf/robots/za_tool_macro.xacro" />
+  <!-- ros2_control parameters-->
+  <xacro:arg name="use_mock_hardware" default="true"/>
+  <xacro:arg name="include_hardware" default="true"/>
+  <xacro:include filename="$(find hydra_description)/urdf/robots/za_tool_macro.xacro"/>
   <xacro:za_tool_macro prefix="$(arg prefix)" tool="$(arg tool)"/>
   <!-- 'world' frame: default pose reference frame -->
@@ -13,11 +16,7 @@
     <child link="$(arg prefix)base_link"/>
   </joint>
-  <!-- Gazebo plugin for ROS Control -->
-  <gazebo>
-    <plugin name="gazebo_ros_control" filename="libgazebo_ros_control.so">
-      <controlPeriod>0.001</controlPeriod>
-      <robotSimType>za_gazebo/ZaHWSim</robotSimType>
-    </plugin>
-    <self_collide>true</self_collide>
-  </gazebo>
+  <xacro:if value="$(arg include_hardware)">
+    <xacro:include filename="$(find za_description)/urdf/za.ros2_control.xacro"/>
+    <xacro:za_ros2_control prefix="$(arg prefix)" use_mock_hardware="$(arg use_mock_hardware)"/>
+  </xacro:if>
 </robot>

File: urdf/tools/typhoon_extruder_macro.xacro (robot description, xacro)
@@ -1,6 +1,6 @@
 <?xml version="1.0"?>
 <robot xmlns:xacro="http://www.ros.org/wiki/xacro">
-    <xacro:property name="tcp_trans" value="0.08613 0.0 -0.159" />
-    <xacro:property name="tcp_rot"  value="0.0 ${pi} 0.0" />
+  <xacro:property name="tcp_trans" value="0.08613 0.0 -0.159" />
+  <xacro:property name="tcp_rot"  value="0.0 ${pi} 0.0" />
 	<xacro:macro name="typhoon_extruder_macro" params="prefix">
 		<!-- link list -->
