Commit message: unify urdf format and remove Gazebo tags

File: urdf/hydra.xacro (robot description, xacro)
@@ -8,14 +8,6 @@
   <link name="world"/>
   <joint name="world-$(arg prefix)hydra_base" type="fixed">
-      <parent link="world"/>
-      <child  link="$(arg prefix)hydra_base"/>
+    <parent link="world"/>
+    <child  link="$(arg prefix)hydra_base"/>
   </joint>
-  <!-- Gazebo plugin for ROS Control -->
-  <gazebo>
-    <plugin name="gazebo_ros_control" filename="libgazebo_ros_control.so">
-      <controlPeriod>0.001</controlPeriod>
-      <robotSimType>hydra_gazebo/HydraHWSim</robotSimType>
-    </plugin>
-    <self_collide>true</self_collide>
-  </gazebo>
 </robot>

File: urdf/hydra_macro.xacro (robot description, xacro)
@@ -1,46 +1,32 @@
 <?xml version="1.0" ?>
 <robot name="hydra" xmlns:xacro="http://www.ros.org/wiki/xacro">
-    <xacro:include filename="$(find hydra_description)/urdf/robots/za_pedestal_macro.xacro"/>
-    <xacro:include filename="$(find hydra_description)/urdf/positioner/positioner_macro.xacro"/>
-    <xacro:macro name="hydra_macro" params="prefix radius tool:='tool0'">
-        <!-- Is the robot being simulated in gazebo? -->
-        <xacro:arg name="gazebo" default="true" />
-        <xacro:za_pedestal_macro prefix="${prefix}rob1_" tool="${tool}"/>
-        <xacro:za_pedestal_macro prefix="${prefix}rob2_" tool="${tool}"/>
-        <xacro:za_pedestal_macro prefix="${prefix}rob3_" tool="${tool}"/>
-        <xacro:positioner_macro prefix="${prefix}"/>
-        <link name="${prefix}hydra_base"/>
-        <joint name="${prefix}hydra_base-rob1_pedestal_base" type="fixed">
-            <origin xyz="-${radius*sin(pi/6)} -${radius*cos(pi/6)}  0" rpy="0 0 ${pi/3}"/>
-            <parent link="${prefix}hydra_base"/>
-            <child  link="${prefix}rob1_pedestal_base"/>
-        </joint>
-        <joint name="${prefix}hydra_base-rob2_pedestal_base" type="fixed">
-            <origin xyz="${radius} 0 0" rpy="0 0 ${pi}"/>
-            <parent link="${prefix}hydra_base"/>
-            <child  link="${prefix}rob2_pedestal_base"/>
-        </joint>
-        <joint name="${prefix}hydra_base-rob3_pedestal_base" type="fixed">
-            <origin xyz="-${radius*sin(pi/6)} ${radius*cos(pi/6)} 0" rpy="0 0 -${pi/3}"/>
-            <parent link="${prefix}hydra_base"/>
-            <child  link="${prefix}rob3_pedestal_base"/>
-        </joint>
-        <joint name="${prefix}hydra_base-$(arg prefix)rotary_table_base" type="fixed">
-            <origin xyz="0 0 0"/>
-            <parent link="${prefix}hydra_base"/>
-            <child  link="${prefix}positioner_stand_base"/>
-        </joint>
-        <xacro:if value="$(arg gazebo)">
-            <transmission name="${prefix}hydra_model">
-              <type>hydra_hw/HydraModelInterface</type>
-              <joint name="${prefix}positioner_joint">
-                <role>positioner</role>
-                <hardwareInterface>hydra_hw/HydraModelInterface</hardwareInterface>
-              </joint>
-              <actuator name="${prefix}_motor_positioner_joint">
-                <hardwareInterface>hydra_hw/HydraModelInterface</hardwareInterface>
-              </actuator>
-            </transmission>
-        </xacro:if>
-    </xacro:macro>
+  <xacro:include filename="$(find hydra_description)/urdf/robots/za_pedestal_macro.xacro"/>
+  <xacro:include filename="$(find hydra_description)/urdf/positioner/positioner_macro.xacro"/>
+  <xacro:macro name="hydra_macro" params="prefix radius tool:='tool0'">
+    <xacro:za_pedestal_macro prefix="${prefix}rob1_" tool="${tool}"/>
+    <xacro:za_pedestal_macro prefix="${prefix}rob2_" tool="${tool}"/>
+    <xacro:za_pedestal_macro prefix="${prefix}rob3_" tool="${tool}"/>
+    <xacro:positioner_macro prefix="${prefix}"/>
+    <link name="${prefix}hydra_base"/>
+    <joint name="${prefix}hydra_base-rob1_pedestal_base" type="fixed">
+      <parent link="${prefix}hydra_base"/>
+      <child  link="${prefix}rob1_pedestal_base"/>
+      <origin xyz="-${radius*sin(pi/6)} -${radius*cos(pi/6)}  0" rpy="0 0 ${pi/3}"/>
+    </joint>
+    <joint name="${prefix}hydra_base-rob2_pedestal_base" type="fixed">
+      <parent link="${prefix}hydra_base"/>
+      <child  link="${prefix}rob2_pedestal_base"/>
+      <origin xyz="${radius} 0 0" rpy="0 0 ${pi}"/>
+    </joint>
+    <joint name="${prefix}hydra_base-rob3_pedestal_base" type="fixed">
+      <parent link="${prefix}hydra_base"/>
+      <child  link="${prefix}rob3_pedestal_base"/>
+      <origin xyz="-${radius*sin(pi/6)} ${radius*cos(pi/6)} 0" rpy="0 0 -${pi/3}"/>
+    </joint>
+    <joint name="${prefix}hydra_base-$(arg prefix)rotary_table_base" type="fixed">
+      <parent link="${prefix}hydra_base"/>
+      <child  link="${prefix}positioner_stand_base"/>
+      <origin xyz="0 0 0"/>
+    </joint>
+  </xacro:macro>
 </robot>

File: urdf/robots/za_pedestal_macro.xacro (robot description, xacro)
@@ -1,30 +1,32 @@
 <?xml version="1.0"?>
 <robot xmlns:xacro="http://www.ros.org/wiki/xacro">
-    <xacro:property name="ped_height" value="0.585" />
-	<xacro:macro name="za_pedestal_macro" params="prefix tool:='tool0'" >
-		<xacro:include filename="$(find hydra_description)/urdf/robots/za_tool_macro.xacro" />
-		<xacro:za_tool_macro prefix="${prefix}" tool="${tool}"/>
-        <link name="${prefix}pedestal_base">
-            <visual>
-                <geometry>
-                    <mesh filename="package://hydra_description/meshes/visual/za_pedestal.dae"/>
-                </geometry>
-            </visual>
-            <collision>
-                <geometry>
-                    <mesh filename="package://hydra_description/meshes/collision/za_pedestal_collision.stl"/>
-                </geometry>
-            </collision>
-        </link>
-		<link name="${prefix}pedestal_top"/>
-        <joint name="${prefix}pedestal_base-${prefix}pedestal_top" type="fixed">
-            <origin rpy="0.0 0.0 0.0" xyz="0 0 ${ped_height}"/>
-            <parent link="${prefix}pedestal_base"/>
-            <child  link="${prefix}pedestal_top"/>
-        </joint>
-        <joint name="${prefix}pedestal_top-${prefix}base_link" type="fixed">
-            <parent link="${prefix}pedestal_top"/>
-            <child  link="${prefix}base_link"/>
-        </joint>
-	</xacro:macro>
+  <xacro:property name="ped_height" value="0.585" />
+  <xacro:macro name="za_pedestal_macro" params="prefix tool:='tool0'" >
+    <xacro:include filename="$(find hydra_description)/urdf/robots/za_tool_macro.xacro" />
+    <xacro:za_tool_macro prefix="${prefix}" tool="${tool}"/>
+    <!-- link list -->
+    <link name="${prefix}pedestal_base">
+      <visual>
+        <geometry>
+          <mesh filename="package://hydra_description/meshes/visual/za_pedestal.dae"/>
+        </geometry>
+      </visual>
+      <collision>
+        <geometry>
+          <mesh filename="package://hydra_description/meshes/collision/za_pedestal_collision.stl"/>
+        </geometry>
+      </collision>
+    </link>
+    <link name="${prefix}pedestal_top"/>
+    <!-- joint list -->
+    <joint name="${prefix}pedestal_base-${prefix}pedestal_top" type="fixed">
+      <parent link="${prefix}pedestal_base"/>
+      <child  link="${prefix}pedestal_top"/>
+      <origin rpy="0.0 0.0 0.0" xyz="0 0 ${ped_height}"/>
+    </joint>
+    <joint name="${prefix}pedestal_top-${prefix}base_link" type="fixed">
+      <parent link="${prefix}pedestal_top"/>
+      <child  link="${prefix}base_link"/>
+    </joint>
+  </xacro:macro>
 </robot>

File: urdf/robots/za_tool.xacro (robot description, xacro)
@@ -8,16 +8,8 @@
   <link name="world" />
   <joint name="world-$(arg prefix)base_link" type="fixed">
+    <parent link="world"/>
+    <child link="$(arg prefix)base_link"/>
     <origin xyz="0 0 0" rpy="0 0 0"/>
     <axis xyz="0 0 1"/>
-    <parent link="world"/>
-    <child link="$(arg prefix)base_link"/>
   </joint>
-  <!-- Gazebo plugin for ROS Control -->
-  <gazebo>
-    <plugin name="gazebo_ros_control" filename="libgazebo_ros_control.so">
-      <controlPeriod>0.001</controlPeriod>
-      <robotSimType>za_gazebo/ZaHWSim</robotSimType>
-    </plugin>
-    <self_collide>true</self_collide>
-  </gazebo>
 </robot>

File: urdf/tools/typhoon_extruder_macro.xacro (robot description, xacro)
@@ -1,37 +1,37 @@
 <?xml version="1.0"?>
 <robot xmlns:xacro="http://www.ros.org/wiki/xacro">
-    <xacro:property name="tcp_trans" value="0.08613 0.0 -0.159" />
-    <xacro:property name="tcp_rot"  value="0.0 ${pi} 0.0" />
-	<xacro:macro name="typhoon_extruder_macro" params="prefix">
-		<!-- link list -->
-		<link name="${prefix}typhoon_extruder">
-			<visual>
-				<geometry>
-					<mesh filename="package://hydra_description/meshes/visual/typhoon_extruder.dae"/>
-				</geometry>
-			</visual>
-			<collision>
-				<geometry>
-					<mesh filename="package://hydra_description/meshes/collision/typhoon_extruder_collision.stl"/>
-				</geometry>
-			</collision>
-			<inertial>
-    			<origin xyz="0.065346 0.000016 -0.031645"/>
-    			<mass value="1.75"/>
-				<inertia ixx="0.006265" ixy="0.000003" ixz="-0.000805" iyy="0.006649" iyz="0.000002" izz="0.001704"/>
-			</inertial>
-		</link>
-		<link name="${prefix}typhoon_extruder_tcp" />
-		<!-- attach extruder to flange -->
-		<joint name="${prefix}extruder_attach_joint" type="fixed">
-			<origin xyz="0 0 0" rpy="0 0 0" />
-			<parent link="${prefix}flange"/>
-			<child link="${prefix}typhoon_extruder"/>
-		</joint>
-		<joint name="${prefix}extruder_extruder_base" type="fixed">
-			<origin xyz="${tcp_trans}" rpy="${tcp_rot}" />
-			<parent link="${prefix}typhoon_extruder"/>
-			<child link="${prefix}typhoon_extruder_tcp"/>
-		</joint>
-	</xacro:macro>
+  <xacro:property name="tcp_trans" value="0.08613 0.0 -0.159" />
+  <xacro:property name="tcp_rot"  value="0.0 ${pi} 0.0" />
+  <xacro:macro name="typhoon_extruder_macro" params="prefix">
+    <!-- link list -->
+    <link name="${prefix}typhoon_extruder">
+      <visual>
+        <geometry>
+          <mesh filename="package://hydra_description/meshes/visual/typhoon_extruder.dae"/>
+        </geometry>
+      </visual>
+      <collision>
+        <geometry>
+          <mesh filename="package://hydra_description/meshes/collision/typhoon_extruder_collision.stl"/>
+        </geometry>
+      </collision>
+      <inertial>
+          <origin xyz="0.065346 0.000016 -0.031645"/>
+          <mass value="1.75"/>
+        <inertia ixx="0.006265" ixy="0.000003" ixz="-0.000805" iyy="0.006649" iyz="0.000002" izz="0.001704"/>
+      </inertial>
+    </link>
+    <link name="${prefix}typhoon_extruder_tcp" />
+    <!-- attach extruder to flange -->
+    <joint name="${prefix}extruder_attach_joint" type="fixed">
+      <parent link="${prefix}flange"/>
+      <child link="${prefix}typhoon_extruder"/>
+      <origin xyz="0 0 0" rpy="0 0 0" />
+    </joint>
+    <joint name="${prefix}extruder_extruder_base" type="fixed">
+      <parent link="${prefix}typhoon_extruder"/>
+      <child link="${prefix}typhoon_extruder_tcp"/>
+      <origin xyz="${tcp_trans}" rpy="${tcp_rot}" />
+    </joint>
+  </xacro:macro>
 </robot>

Commit message: unify urdf format and remove Gazebo tags

File: urdf/hydra.xacro (robot description, xacro)
@@ -11,11 +11,3 @@
       <child  link="$(arg prefix)hydra_base"/>
   </joint>
-  <!-- Gazebo plugin for ROS Control -->
-  <gazebo>
-    <plugin name="gazebo_ros_control" filename="libgazebo_ros_control.so">
-      <controlPeriod>0.001</controlPeriod>
-      <robotSimType>hydra_gazebo/HydraHWSim</robotSimType>
-    </plugin>
-    <self_collide>true</self_collide>
-  </gazebo>
 </robot>

File: urdf/hydra_macro.xacro (robot description, xacro)
@@ -4,6 +4,4 @@
     <xacro:include filename="$(find hydra_description)/urdf/robots/za_positioner_macro.xacro"/>
     <xacro:macro name="hydra_macro" params="prefix radius tool:='tool0'">
-      <!-- Is the robot being simulated in gazebo? -->
-      <xacro:arg name="gazebo" default="true" />
       <xacro:za_pedestal_macro prefix="${prefix}rob1_" tool="${tool}"/>
       <xacro:za_pedestal_macro prefix="${prefix}rob2_" tool="${tool}"/>
@@ -25,16 +23,4 @@
         <child  link="${prefix}rob3_base_link"/>
       </joint>
-      <xacro:if value="$(arg gazebo)">
-        <transmission name="${prefix}hydra_model">
-          <type>hydra_hw/HydraModelInterface</type>
-          <joint name="${prefix}positioner_joint">
-            <role>positioner</role>
-            <hardwareInterface>hydra_hw/HydraModelInterface</hardwareInterface>
-          </joint>
-          <actuator name="${prefix}_motor_positioner_joint">
-            <hardwareInterface>hydra_hw/HydraModelInterface</hardwareInterface>
-          </actuator>
-        </transmission>
-      </xacro:if>
     </xacro:macro>
   </robot>

File: urdf/robots/za_pedestal_macro.xacro (robot description, xacro)
@@ -1,30 +1,32 @@
 <?xml version="1.0"?>
 <robot xmlns:xacro="http://www.ros.org/wiki/xacro">
-    <xacro:property name="ped_height" value="0.585" />
-	<xacro:macro name="za_pedestal_macro" params="prefix tool:='tool0'" >
-		<xacro:include filename="$(find hydra_description)/urdf/robots/za_tool_macro.xacro" />
-		<xacro:za_tool_macro prefix="${prefix}" tool="${tool}"/>
-        <link name="${prefix}pedestal_base">
-            <visual>
-                <geometry>
-                    <mesh filename="package://hydra_description/meshes/visual/za_pedestal.dae"/>
-                </geometry>
-            </visual>
-            <collision>
-                <geometry>
-                    <mesh filename="package://hydra_description/meshes/collision/za_pedestal_collision.stl"/>
-                </geometry>
-            </collision>
-        </link>
-		<link name="${prefix}pedestal_top"/>
-        <joint name="${prefix}pedestal_base-${prefix}pedestal_top" type="fixed">
-            <origin rpy="0.0 0.0 0.0" xyz="0 0 ${ped_height}"/>
-            <parent link="${prefix}pedestal_base"/>
-            <child  link="${prefix}pedestal_top"/>
-        </joint>
-        <joint name="${prefix}pedestal_top-${prefix}base_link" type="fixed">
-            <parent link="${prefix}pedestal_top"/>
-            <child  link="${prefix}base_link"/>
-        </joint>
-	</xacro:macro>
+  <xacro:property name="ped_height" value="0.585" />
+  <xacro:macro name="za_pedestal_macro" params="prefix tool:='tool0'" >
+    <xacro:include filename="$(find hydra_description)/urdf/robots/za_tool_macro.xacro" />
+    <xacro:za_tool_macro prefix="${prefix}" tool="${tool}"/>
+    <!-- link list -->
+    <link name="${prefix}pedestal_base">
+      <visual>
+        <geometry>
+          <mesh filename="package://hydra_description/meshes/visual/za_pedestal.dae"/>
+        </geometry>
+      </visual>
+      <collision>
+        <geometry>
+          <mesh filename="package://hydra_description/meshes/collision/za_pedestal_collision.stl"/>
+        </geometry>
+      </collision>
+      </link>
+    <link name="${prefix}pedestal_top"/>
+    <!-- joint list -->
+    <joint name="${prefix}pedestal_base-${prefix}pedestal_top" type="fixed">
+      <parent link="${prefix}pedestal_base"/>
+      <child  link="${prefix}pedestal_top"/>
+      <origin rpy="0.0 0.0 0.0" xyz="0 0 ${ped_height}"/>
+    </joint>
+    <joint name="${prefix}pedestal_top-${prefix}base_link" type="fixed">
+      <parent link="${prefix}pedestal_top"/>
+      <child  link="${prefix}base_link"/>
+    </joint>
+  </xacro:macro>
 </robot>

File: urdf/robots/za_positioner.xacro (robot description, xacro)
@@ -12,11 +12,3 @@
     <child link="$(arg prefix)base_link"/>
   </joint>
-  <!-- Gazebo plugin for ROS Control -->
-  <gazebo>
-    <plugin name="gazebo_ros_control" filename="libgazebo_ros_control.so">
-      <controlPeriod>0.001</controlPeriod>
-      <robotSimType>za_gazebo/ZaHWSim</robotSimType>
-    </plugin>
-    <self_collide>true</self_collide>
-  </gazebo>
 </robot>

File: urdf/robots/za_positioner_macro.xacro (robot description, xacro)
@@ -1,7 +1,7 @@
 <?xml version="1.0"?>
 <robot xmlns:xacro="http://www.ros.org/wiki/xacro">
-	<xacro:macro name="za_positioner_macro" params="prefix" >
-		<xacro:include filename="$(find za_description)/urdf/za_macro.xacro" />
-		<xacro:za_macro prefix="${prefix}" />
+  <xacro:macro name="za_positioner_macro" params="prefix" >
+    <xacro:include filename="$(find za_description)/urdf/za_macro.xacro" />
+    <xacro:za_macro prefix="${prefix}" />
     <!-- link list -->
     <link name="${prefix}positioner_base">
@@ -25,12 +25,12 @@
     <!-- joint list -->
     <joint name="${prefix}flange_positioner_base" type="fixed">
-      <origin rpy="0 ${pi/2} 0" xyz="0 0 0"/>
       <parent link="${prefix}flange"/>
       <child link="${prefix}positioner_base"/>
+      <origin rpy="0 ${pi/2} 0" xyz="0 0 0"/>
     </joint>
     <joint name="${prefix}positioner_tcp_joint" type="fixed">
-      <origin rpy="0.0 0.0 0.0" xyz="0 0 0.03175"/>
       <parent link="${prefix}positioner_base"/>
       <child link="${prefix}positioner"/>
+      <origin rpy="0.0 0.0 0.0" xyz="0 0 0.03175"/>
     </joint>
   </xacro:macro>

File: urdf/robots/za_tool.xacro (robot description, xacro)
@@ -13,11 +13,3 @@
     <child link="$(arg prefix)base_link"/>
   </joint>
-  <!-- Gazebo plugin for ROS Control -->
-  <gazebo>
-    <plugin name="gazebo_ros_control" filename="libgazebo_ros_control.so">
-      <controlPeriod>0.001</controlPeriod>
-      <robotSimType>za_gazebo/ZaHWSim</robotSimType>
-    </plugin>
-    <self_collide>true</self_collide>
-  </gazebo>
 </robot>

File: urdf/tools/typhoon_extruder_macro.xacro (robot description, xacro)
@@ -1,37 +1,37 @@
 <?xml version="1.0"?>
 <robot xmlns:xacro="http://www.ros.org/wiki/xacro">
-    <xacro:property name="tcp_trans" value="0.08613 0.0 -0.159" />
-    <xacro:property name="tcp_rot"  value="0.0 ${pi} 0.0" />
-	<xacro:macro name="typhoon_extruder_macro" params="prefix">
-		<!-- link list -->
-		<link name="${prefix}typhoon_extruder">
-			<visual>
-				<geometry>
-					<mesh filename="package://hydra_description/meshes/visual/typhoon_extruder.dae"/>
-				</geometry>
-			</visual>
-			<collision>
-				<geometry>
-					<mesh filename="package://hydra_description/meshes/collision/typhoon_extruder_collision.stl"/>
-				</geometry>
-			</collision>
-			<inertial>
-    			<origin xyz="0.065346 0.000016 -0.031645"/>
-    			<mass value="1.75"/>
-				<inertia ixx="0.006265" ixy="0.000003" ixz="-0.000805" iyy="0.006649" iyz="0.000002" izz="0.001704"/>
-			</inertial>
-		</link>
-		<link name="${prefix}typhoon_extruder_tcp" />
-		<!-- attach extruder to flange -->
-		<joint name="${prefix}extruder_attach_joint" type="fixed">
-			<origin xyz="0 0 0" rpy="0 0 0" />
-			<parent link="${prefix}flange"/>
-			<child link="${prefix}typhoon_extruder"/>
-		</joint>
-		<joint name="${prefix}extruder_extruder_base" type="fixed">
-			<origin xyz="${tcp_trans}" rpy="${tcp_rot}" />
-			<parent link="${prefix}typhoon_extruder"/>
-			<child link="${prefix}typhoon_extruder_tcp"/>
-		</joint>
-	</xacro:macro>
+  <xacro:property name="tcp_trans" value="0.08613 0.0 -0.159" />
+  <xacro:property name="tcp_rot"  value="0.0 ${pi} 0.0" />
+  <xacro:macro name="typhoon_extruder_macro" params="prefix">
+    <!-- link list -->
+    <link name="${prefix}typhoon_extruder">
+      <visual>
+        <geometry>
+          <mesh filename="package://hydra_description/meshes/visual/typhoon_extruder.dae"/>
+        </geometry>
+      </visual>
+      <collision>
+        <geometry>
+          <mesh filename="package://hydra_description/meshes/collision/typhoon_extruder_collision.stl"/>
+        </geometry>
+      </collision>
+      <inertial>
+          <origin xyz="0.065346 0.000016 -0.031645"/>
+          <mass value="1.75"/>
+        <inertia ixx="0.006265" ixy="0.000003" ixz="-0.000805" iyy="0.006649" iyz="0.000002" izz="0.001704"/>
+      </inertial>
+    </link>
+    <link name="${prefix}typhoon_extruder_tcp" />
+    <!-- attach extruder to flange -->
+    <joint name="${prefix}extruder_attach_joint" type="fixed">
+      <origin xyz="0 0 0" rpy="0 0 0" />
+      <parent link="${prefix}flange"/>
+      <child link="${prefix}typhoon_extruder"/>
+    </joint>
+    <joint name="${prefix}extruder_extruder_base" type="fixed">
+      <origin xyz="${tcp_trans}" rpy="${tcp_rot}" />
+      <parent link="${prefix}typhoon_extruder"/>
+      <child link="${prefix}typhoon_extruder_tcp"/>
+    </joint>
+  </xacro:macro>
 </robot>
