Commit message: reverse pedestal chain direction

File: urdf/hydra.xacro (robot description, xacro)
@@ -8,10 +8,5 @@
   <xacro:arg name="include_hardware" default="true"/>
   <xacro:include filename="$(find hydra_description)/urdf/hydra_macro.xacro"/>
-  <xacro:hydra_macro prefix="$(arg prefix)"
-    radius="${radius}"
-    tool="${tool}"
-    include_hardware="$(arg include_hardware)"
-    use_mock_hardware="$(arg use_mock_hardware)"
-  />
+  <xacro:hydra_macro prefix="$(arg prefix)" radius="${radius}" tool="${tool}"/>
   <link name="world"/>
   <joint name="world-$(arg prefix)hydra_base" type="fixed">
@@ -21,7 +16,12 @@
   <link name="work_object"/>
   <joint name="world-$(arg prefix)work_object" type="fixed">
-    <origin xyz="0 0 0.8" rpy="0 0 0"/>
+    <origin xyz="0 0 0" rpy="0 0 0"/>
     <parent link="world"/>
     <child  link="$(arg prefix)work_object"/>
   </joint>
+  <xacro:if value="$(arg include_hardware)">
+    <xacro:include filename="$(find za_description)/urdf/za.ros2_control.xacro"/>
+    <xacro:za_ros2_control prefix="$(arg prefix)rob1_" use_mock_hardware="$(arg use_mock_hardware)"/>
+    <xacro:za_ros2_control prefix="$(arg prefix)rob2_" use_mock_hardware="$(arg use_mock_hardware)"/>
+  </xacro:if>
 </robot>

File: urdf/hydra_macro.xacro (robot description, xacro)
@@ -2,28 +2,23 @@
 <robot name="hydra" xmlns:xacro="http://www.ros.org/wiki/xacro">
   <xacro:include filename="$(find hydra_description)/urdf/robots/za_pedestal_macro.xacro"/>
-  <xacro:macro name="hydra_macro" params="
-    prefix
-    radius
-    tool:='tool0'
-    include_hardware:=false
-    use_mock_hardware:=true">
+  <xacro:macro name="hydra_macro" params="prefix radius tool:='tool0'">
+    <xacro:property name="rob1_base_origin" value="0 -${radius} 0"/>
+    <xacro:property name="rob1_base_rot" value="0 0 ${pi/2}"/>
+    <xacro:property name="rob2_base_origin" value="0 ${radius} 0"/>
+    <xacro:property name="rob2_base_rot" value="0 0 -${pi/2}"/>
     <xacro:za_pedestal_macro prefix="${prefix}rob1_" tool="${tool}"/>
     <xacro:za_pedestal_macro prefix="${prefix}rob2_" tool="${tool}"/>
     <link name="${prefix}hydra_base"/>
-    <joint name="${prefix}hydra_base-rob1_pedestal_base" type="fixed">
-      <origin xyz="0 -${radius}  0" rpy="0 0 ${pi/2}"/>
-      <parent link="${prefix}world"/>
-      <child  link="${prefix}rob1_pedestal_base"/>
+    <!-- joint list -->
+    <joint name="${prefix}hydra_base-rob1_base_link" type="fixed">
+      <parent link="${prefix}hydra_base"/>
+      <child  link="${prefix}rob1_base_link"/>
+      <origin xyz="${rob1_base_origin}" rpy="${rob1_base_rot}"/>
     </joint>
-    <joint name="${prefix}hydra_base-rob2_pedestal_base" type="fixed">
-      <origin xyz="0 ${radius} 0" rpy="0 0 -${pi/2}"/>
-      <parent link="${prefix}world"/>
-      <child  link="${prefix}rob2_pedestal_base"/>
+    <joint name="${prefix}hydra_base-rob2_base_link" type="fixed">
+      <parent link="${prefix}hydra_base"/>
+      <child  link="${prefix}rob2_base_link"/>
+      <origin xyz="${rob2_base_origin}" rpy="${rob2_base_rot}"/>
     </joint>
-    <xacro:if value="${include_hardware}">
-      <xacro:include filename="$(find za_description)/urdf/za.ros2_control.xacro"/>
-      <xacro:za_ros2_control prefix="${prefix}rob1_" use_mock_hardware="${use_mock_hardware}"/>
-      <xacro:za_ros2_control prefix="${prefix}rob2_" use_mock_hardware="${use_mock_hardware}"/>
-    </xacro:if>
   </xacro:macro>
 </robot>

File: urdf/robots/za_pedestal_macro.xacro (robot description, xacro)
@@ -31,17 +31,17 @@
     </link>
     <link name="${prefix}pedestal_top"/>
-    <joint name="${prefix}pedestal_base-${prefix}pedestal" type="fixed">
-      <origin rpy="0.0 0.0 0.0" xyz="0 0 ${base_height}"/>
-      <parent link="${prefix}pedestal_base"/>
+    <joint name="${prefix}base_link-${prefix}pedestal_top" type="fixed">
+      <parent link="${prefix}base_link"/>
+      <child  link="${prefix}pedestal_top"/>
+    </joint>
+    <joint name="${prefix}pedestal_top-${prefix}pedestal" type="fixed">
+      <origin rpy="0.0 0.0 0.0" xyz="0 0 ${-ped_height}"/>
+      <parent link="${prefix}pedestal_top"/>
       <child  link="${prefix}pedestal"/>
     </joint>
-    <joint name="${prefix}pedestal-${prefix}pedestal_top" type="fixed">
-      <origin rpy="0.0 0.0 0.0" xyz="0 0 ${ped_height}"/>
+    <joint name="${prefix}pedestal-${prefix}pedestal_base" type="fixed">
+      <origin rpy="0.0 0.0 0.0" xyz="0 0 ${-base_height}"/>
       <parent link="${prefix}pedestal"/>
-      <child  link="${prefix}pedestal_top"/>
-    </joint>
-    <joint name="${prefix}pedestal_top-${prefix}base_link" type="fixed">
-      <parent link="${prefix}pedestal_top"/>
-      <child  link="${prefix}base_link"/>
+      <child  link="${prefix}pedestal_base"/>
     </joint>
   </xacro:macro>

Commit message: fix position of work object frame

File: urdf/hydra.xacro (robot description, xacro)
@@ -8,11 +8,12 @@
   <link name="world"/>
   <joint name="world-$(arg prefix)hydra_base" type="fixed">
+    <origin xyz="0 0 0.785" rpy="0 0 0"/>
     <parent link="world"/>
     <child  link="$(arg prefix)hydra_base"/>
   </joint>
   <link name="work_object"/>
-  <joint name="world-$(arg prefix)work_object" type="fixed">
-    <origin xyz="0 0 0.8" rpy="0 0 0"/>
-    <parent link="world"/>
+  <joint name="$(arg prefix)hydra_base-$(arg prefix)work_object" type="fixed">
+    <origin xyz="0 0 0" rpy="0 0 0"/>
+    <parent link="$(arg prefix)hydra_base"/>
     <child  link="$(arg prefix)work_object"/>
   </joint>

Commit message: use yaml files to define tool, base, and wobj data

File: urdf/hydra.xacro (robot description, xacro)
@@ -2,8 +2,15 @@
 <robot name="hydra" xmlns:xacro="http://www.ros.org/wiki/xacro">
   <xacro:arg name="prefix" default=""/>
-  <xacro:property name="radius" value="0.75"/>
-  <xacro:property name="tool" default="typhoon_extruder" />
+  <xacro:arg name="tool"   default="typhoon_extruder"/>
+  <xacro:property name="tool_parameters_file"  value="$(find hydra_description)/config/tool_parameters.yaml"/>
+  <xacro:property name="kinematic_parameters_file" value="$(find hydra_description)/config/kinematic_parameters.yaml"/>
   <xacro:include filename="$(find hydra_description)/urdf/hydra_macro.xacro"/>
-  <xacro:hydra_macro prefix="$(arg prefix)" radius="${radius}" tool="${tool}"/>
+  <xacro:hydra_macro
+    prefix="$(arg prefix)"
+    tool_parameters_file="${tool_parameters_file}"
+    kinematic_parameters_file="${kinematic_parameters_file}"
+    rob1_tool="$(arg tool)"
+    rob2_tool="$(arg tool)"
+  />
   <link name="world"/>
   <joint name="world-$(arg prefix)hydra_base" type="fixed">
@@ -12,9 +19,3 @@
     <child  link="$(arg prefix)hydra_base"/>
   </joint>
-  <link name="work_object"/>
-  <joint name="$(arg prefix)hydra_base-$(arg prefix)work_object" type="fixed">
-    <origin xyz="0 0 0" rpy="0 0 0"/>
-    <parent link="$(arg prefix)hydra_base"/>
-    <child  link="$(arg prefix)work_object"/>
-  </joint>
 </robot>

File: urdf/hydra_macro.xacro (robot description, xacro)
@@ -2,22 +2,53 @@
 <robot name="hydra" xmlns:xacro="http://www.ros.org/wiki/xacro">
   <xacro:include filename="$(find hydra_description)/urdf/robots/za_pedestal_macro.xacro"/>
-  <xacro:macro name="hydra_macro" params="prefix radius tool:='tool0'">
-    <xacro:property name="rob1_base_origin" value="0 -${radius} 0"/>
-    <xacro:property name="rob1_base_rot" value="0 0 ${pi/2}"/>
-    <xacro:property name="rob2_base_origin" value="0 ${radius} 0"/>
-    <xacro:property name="rob2_base_rot" value="0 0 -${pi/2}"/>
-    <xacro:za_pedestal_macro prefix="${prefix}rob1_" tool="${tool}"/>
-    <xacro:za_pedestal_macro prefix="${prefix}rob2_" tool="${tool}"/>
+  <xacro:macro name="hydra_macro" params="
+    prefix
+    tool_parameters_file
+    kinematic_parameters_file
+    rob1_tool:='tool0'
+    rob2_tool:='tool0'"
+  >
+    <!-- Load end effector and work object parameters -->
+    <xacro:property name="tool_data" value="${xacro.load_yaml(tool_parameters_file)}"/>
+    <xacro:property name="kin_data" value="${xacro.load_yaml(kinematic_parameters_file)}"/>
+    <xacro:property name="wobj_data" value="${kin_data['whiteboard']}"/>
+    <xacro:property name="wobj_xyz" value="${wobj_data['x']} ${wobj_data['y']} ${wobj_data['z']}"/>
+    <xacro:property name="wobj_rpy" value="${wobj_data['roll']} ${wobj_data['pitch']} ${wobj_data['yaw']}"/>
+    <xacro:property name="rob1_base_data" value="${kin_data['rob1_base']}"/>
+    <xacro:property name="rob1_base_xyz" value="${rob1_base_data['x']} ${rob1_base_data['y']} ${rob1_base_data['z']}"/>
+    <xacro:property name="rob1_base_rpy" value="${rob1_base_data['roll']} ${rob1_base_data['pitch']} ${rob1_base_data['yaw']}"/>
+    <xacro:property name="rob2_base_data" value="${kin_data['rob2_base']}"/>
+    <xacro:property name="rob2_base_xyz" value="${rob2_base_data['x']} ${rob2_base_data['y']} ${rob2_base_data['z']}"/>
+    <xacro:property name="rob2_base_rpy" value="${rob2_base_data['roll']} ${rob2_base_data['pitch']} ${rob2_base_data['yaw']}"/>
+    <xacro:za_pedestal_macro prefix="${prefix}rob1_" tool_data="${tool_data['rob1']}" tool="${rob1_tool}"/>
+    <xacro:za_pedestal_macro prefix="${prefix}rob2_" tool_data="${tool_data['rob2']}" tool="${rob2_tool}"/>
     <link name="${prefix}hydra_base"/>
+    <link name="${prefix}work_object">
+      <visual>
+        <geometry>
+          <mesh filename="package://hydra_description/meshes/visual/whiteboard.dae"/>
+        </geometry>
+      </visual>
+      <collision>
+        <geometry>
+          <mesh filename="package://hydra_description/meshes/collision/whiteboard_collision.stl"/>
+        </geometry>
+      </collision>
+    </link>
     <!-- joint list -->
     <joint name="${prefix}hydra_base-rob1_base_link" type="fixed">
       <parent link="${prefix}hydra_base"/>
       <child  link="${prefix}rob1_base_link"/>
-      <origin xyz="${rob1_base_origin}" rpy="${rob1_base_rot}"/>
+      <origin xyz="${rob1_base_xyz}" rpy="${rob1_base_rpy}"/>
     </joint>
     <joint name="${prefix}hydra_base-rob2_base_link" type="fixed">
       <parent link="${prefix}hydra_base"/>
       <child  link="${prefix}rob2_base_link"/>
-      <origin xyz="${rob2_base_origin}" rpy="${rob2_base_rot}"/>
+      <origin xyz="${rob2_base_xyz}" rpy="${rob2_base_rpy}"/>
+    </joint>
+    <joint name="${prefix}hydra_base-${prefix}work_object" type="fixed">
+      <parent link="${prefix}hydra_base"/>
+      <child  link="${prefix}work_object"/>
+      <origin xyz="${wobj_xyz}" rpy="${wobj_rpy}"/>
     </joint>
   </xacro:macro>

File: urdf/robots/za_pedestal.xacro (robot description, xacro)
@@ -3,5 +3,7 @@
   <xacro:arg name="prefix" default="" />
   <xacro:arg name="tool" default="typhoon_extruder" />
+  <xacro:property name="tool_parameters_file" value="$(find hydra_description)/config/tool_parameters.yaml"/>
+  <xacro:property name="tool_data" value="${xacro.load_yaml(tool_parameters_file)}"/>
   <xacro:include filename="$(find hydra_description)/urdf/robots/za_pedestal_macro.xacro" />
-  <xacro:za_pedestal_macro prefix="$(arg prefix)" tool="$(arg tool)"/>
+  <xacro:za_pedestal_macro prefix="$(arg prefix)" tool_data="${tool_data['rob1']}" tool="$(arg tool)"/>
 </robot>

File: urdf/robots/za_pedestal_macro.xacro (robot description, xacro)
@@ -3,7 +3,7 @@
   <xacro:property name="ped_height" value="0.585"/>
   <xacro:property name="base_height" value="0.2"/>
-  <xacro:macro name="za_pedestal_macro" params="prefix tool:='tool0'" >
-    <xacro:include filename="$(find hydra_description)/urdf/robots/za_tool_macro.xacro" />
-    <xacro:za_tool_macro prefix="${prefix}" tool="${tool}"/>
+  <xacro:macro name="za_pedestal_macro" params="prefix tool_data tool:='tool0'">
+    <xacro:include filename="$(find hydra_description)/urdf/robots/za_tool_macro.xacro"/>
+    <xacro:za_tool_macro prefix="${prefix}" tool_data="${tool_data}" tool="${tool}"/>
     <link name="${prefix}pedestal_base">
       <visual>
@@ -14,5 +14,5 @@
       <collision>
         <geometry>
-          <mesh filename="package://hydra_description/meshes/collision/optical_table.stl"/>
+          <mesh filename="package://hydra_description/meshes/collision/hframe_base_collision.stl"/>
         </geometry>
       </collision>

File: urdf/robots/za_tool.xacro (robot description, xacro)
@@ -3,6 +3,8 @@
   <xacro:arg name="prefix" default="" />
   <xacro:arg name="tool" default="typhoon_extruder" />
+  <xacro:property name="tool_parameters_file" value="$(find hydra_description)/config/tool_parameters.yaml"/>
+  <xacro:property name="tool_data" value="${xacro.load_yaml(tool_parameters_file)}"/>
   <xacro:include filename="$(find hydra_description)/urdf/robots/za_tool_macro.xacro" />
-  <xacro:za_tool_macro prefix="$(arg prefix)" tool="$(arg tool)"/>
+  <xacro:za_tool_macro prefix="$(arg prefix)" tool_data="${tool_data['rob1']}" tool="$(arg tool)"/>
   <!-- 'world' frame: default pose reference frame -->
   <link name="world" />

File: urdf/robots/za_tool_macro.xacro (robot description, xacro)
@@ -1,11 +1,14 @@
 <?xml version="1.0"?>
 <robot xmlns:xacro="http://www.ros.org/wiki/xacro">
-  <xacro:macro name="za_tool_macro" params="prefix tool:='tool0'" >
+  <xacro:macro name="za_tool_macro" params="prefix tool_data tool:='tool0'">
     <xacro:include filename="$(find za_description)/urdf/za_macro.xacro" />
-    <xacro:za_macro prefix="${prefix}" />
-    <xml:property name="var" value="typhoon_extruder"/>
+    <xacro:za_macro prefix="${prefix}"/>
     <xacro:if value="${tool == 'typhoon_extruder'}">
       <xacro:include filename="$(find hydra_description)/urdf/tools/typhoon_extruder_macro.xacro" />
-      <xacro:typhoon_extruder_macro prefix="${prefix}" />
+      <xacro:typhoon_extruder_macro prefix="${prefix}" tool_data="${tool_data['typhoon_extruder']}"/>
+    </xacro:if>
+    <xacro:if value="${tool == 'marker_tool'}">
+      <xacro:include filename="$(find hydra_description)/urdf/tools/marker_tool_macro.xacro" />
+      <xacro:marker_tool_macro prefix="${prefix}" tool_data="${tool_data['marker_tool']}"/>
     </xacro:if>
   </xacro:macro>

File: urdf/tools/typhoon_extruder_macro.xacro (robot description, xacro)
@@ -1,7 +1,7 @@
 <?xml version="1.0"?>
 <robot xmlns:xacro="http://www.ros.org/wiki/xacro">
-  <xacro:property name="tcp_trans" value="0.08613 0.0 -0.159" />
-  <xacro:property name="tcp_rot"  value="0.0 ${pi} 0.0" />
-  <xacro:macro name="typhoon_extruder_macro" params="prefix">
+  <xacro:macro name="typhoon_extruder_macro" params="prefix tool_data">
+    <xacro:property name="tcp_xyz" value="${tool_data['x']} ${tool_data['y']} ${tool_data['z']}"/>
+    <xacro:property name="tcp_rpy" value="${tool_data['roll']} ${tool_data['pitch']} ${tool_data['yaw']}"/>
     <!-- link list -->
     <link name="${prefix}typhoon_extruder">
@@ -27,5 +27,5 @@
       <parent link="${prefix}typhoon_extruder"/>
       <child link="${prefix}typhoon_extruder_tcp"/>
-      <origin xyz="${tcp_trans}" rpy="${tcp_rot}" />
+      <origin xyz="${tcp_xyz}" rpy="${tcp_rpy}" />
     </joint>
   </xacro:macro>

Commit message: swap robots and redefine whiteboard frame location

File: urdf/hydra.xacro (robot description, xacro)
@@ -3,5 +3,5 @@
   <xacro:arg name="prefix" default=""/>
   <xacro:arg name="tool"   default="typhoon_extruder"/>
-  <xacro:property name="tool_parameters_file"  value="$(find hydra_description)/config/tool_parameters.yaml"/>
+  <xacro:property name="tool_parameters_file" value="$(find hydra_description)/config/tool_parameters.yaml"/>
   <xacro:property name="kinematic_parameters_file" value="$(find hydra_description)/config/kinematic_parameters.yaml"/>
   <xacro:include filename="$(find hydra_description)/urdf/hydra_macro.xacro"/>

File: urdf/robots/za_pedestal.xacro (robot description, xacro)
@@ -2,8 +2,15 @@
 <robot name="za" xmlns:xacro="http://www.ros.org/wiki/xacro">
   <xacro:arg name="prefix" default="" />
-  <xacro:arg name="tool" default="typhoon_extruder" />
+  <xacro:arg name="tool" default="typhoon_extruder"/>
   <xacro:property name="tool_parameters_file" value="$(find hydra_description)/config/tool_parameters.yaml"/>
   <xacro:property name="tool_data" value="${xacro.load_yaml(tool_parameters_file)}"/>
   <xacro:include filename="$(find hydra_description)/urdf/robots/za_pedestal_macro.xacro" />
   <xacro:za_pedestal_macro prefix="$(arg prefix)" tool_data="${tool_data['rob1']}" tool="$(arg tool)"/>
+  <!-- 'world' frame: default pose reference frame -->
+  <link name="world" />
+  <joint name="world-$(arg prefix)base_link" type="fixed">
+    <parent link="world"/>
+    <child link="$(arg prefix)base_link"/>
+    <origin xyz="0 0 0" rpy="0 0 0"/>
+  </joint>
 </robot>

File: urdf/robots/za_tool.xacro (robot description, xacro)
@@ -2,5 +2,5 @@
 <robot name="za" xmlns:xacro="http://www.ros.org/wiki/xacro">
   <xacro:arg name="prefix" default="" />
-  <xacro:arg name="tool" default="typhoon_extruder" />
+  <xacro:arg name="tool" default="typhoon_extruder"/>
   <xacro:property name="tool_parameters_file" value="$(find hydra_description)/config/tool_parameters.yaml"/>
   <xacro:property name="tool_data" value="${xacro.load_yaml(tool_parameters_file)}"/>
