Commit message: use yaml files to define tool, base, and wobj data

File: urdf/hydra.xacro (robot description, xacro)
@@ -2,8 +2,16 @@
 <robot name="hydra" xmlns:xacro="http://www.ros.org/wiki/xacro">
   <xacro:arg name="prefix" default=""/>
-  <xacro:property name="radius" value="0.95" />
-  <xacro:property name="tool" default="typhoon_extruder" />
+  <xacro:arg name="tool" default="typhoon_extruder"/>
+  <xacro:property name="tool_parameters_file" value="$(find hydra_description)/config/tool_parameters.yaml"/>
+  <xacro:property name="kinematic_parameters_file" value="$(find hydra_description)/config/kinematic_parameters.yaml"/>
   <xacro:include filename="$(find hydra_description)/urdf/hydra_macro.xacro"/>
-  <xacro:hydra_macro prefix="$(arg prefix)" radius="${radius}" tool="${tool}"/>
+  <xacro:hydra_macro
+    prefix="$(arg prefix)"
+    tool_parameters_file="${tool_parameters_file}"
+    kinematic_parameters_file="${kinematic_parameters_file}"
+    rob1_tool="$(arg tool)"
+    rob2_tool="$(arg tool)"
+    rob3_tool="$(arg tool)"
+  />
   <link name="world"/>
   <joint name="world-$(arg prefix)hydra_base" type="fixed">

File: urdf/hydra_macro.xacro (robot description, xacro)
@@ -3,29 +3,51 @@
   <xacro:include filename="$(find hydra_description)/urdf/robots/za_pedestal_macro.xacro"/>
   <xacro:include filename="$(find hydra_description)/urdf/positioner/positioner_macro.xacro"/>
-  <xacro:macro name="hydra_macro" params="prefix radius tool:='tool0'">
-    <xacro:za_pedestal_macro prefix="${prefix}rob1_" tool="${tool}"/>
-    <xacro:za_pedestal_macro prefix="${prefix}rob2_" tool="${tool}"/>
-    <xacro:za_pedestal_macro prefix="${prefix}rob3_" tool="${tool}"/>
+  <xacro:macro name="hydra_macro" params="
+    prefix
+    tool_parameters_file
+    kinematic_parameters_file
+    rob1_tool:='tool0'
+    rob2_tool:='tool0'
+    rob3_tool:='tool0'
+  ">
+    <!-- Load kinematics and tool parameters -->
+    <xacro:property name="tool_data" value="${xacro.load_yaml(tool_parameters_file)}"/>
+    <xacro:property name="kin_data" value="${xacro.load_yaml(kinematic_parameters_file)}"/>
+    <xacro:property name="wobj_data" value="${kin_data['positioner']}"/>
+    <xacro:property name="wobj_xyz" value="${wobj_data['x']} ${wobj_data['y']} ${wobj_data['z']}"/>
+    <xacro:property name="wobj_rpy" value="${wobj_data['roll']} ${wobj_data['pitch']} ${wobj_data['yaw']}"/>
+    <xacro:property name="rob1_base_data" value="${kin_data['rob1_base']}"/>
+    <xacro:property name="rob1_base_xyz" value="${rob1_base_data['x']} ${rob1_base_data['y']} ${rob1_base_data['z']}"/>
+    <xacro:property name="rob1_base_rpy" value="${rob1_base_data['roll']} ${rob1_base_data['pitch']} ${rob1_base_data['yaw']}"/>
+    <xacro:property name="rob2_base_data" value="${kin_data['rob2_base']}"/>
+    <xacro:property name="rob2_base_xyz" value="${rob2_base_data['x']} ${rob2_base_data['y']} ${rob2_base_data['z']}"/>
+    <xacro:property name="rob2_base_rpy" value="${rob2_base_data['roll']} ${rob2_base_data['pitch']} ${rob2_base_data['yaw']}"/>
+    <xacro:property name="rob3_base_data" value="${kin_data['rob3_base']}"/>
+    <xacro:property name="rob3_base_xyz" value="${rob3_base_data['x']} ${rob3_base_data['y']} ${rob3_base_data['z']}"/>
+    <xacro:property name="rob3_base_rpy" value="${rob3_base_data['roll']} ${rob3_base_data['pitch']} ${rob3_base_data['yaw']}"/>
+    <xacro:za_pedestal_macro prefix="${prefix}rob1_" tool_data="${tool_data['rob1']}" tool="${rob1_tool}"/>
+    <xacro:za_pedestal_macro prefix="${prefix}rob2_" tool_data="${tool_data['rob2']}" tool="${rob2_tool}"/>
+    <xacro:za_pedestal_macro prefix="${prefix}rob3_" tool_data="${tool_data['rob3']}" tool="${rob3_tool}"/>
     <xacro:positioner_macro prefix="${prefix}"/>
     <link name="${prefix}hydra_base"/>
-    <joint name="${prefix}hydra_base-rob1_pedestal_base" type="fixed">
+    <joint name="${prefix}hydra_base-rob1_base_link" type="fixed">
       <parent link="${prefix}hydra_base"/>
-      <child  link="${prefix}rob1_pedestal_base"/>
-      <origin xyz="-${radius*sin(pi/6)} -${radius*cos(pi/6)}  0" rpy="0 0 ${pi/3}"/>
+      <child  link="${prefix}rob1_base_link"/>
+      <origin xyz="${rob1_base_xyz}" rpy="${rob1_base_rpy}"/>
     </joint>
-    <joint name="${prefix}hydra_base-rob2_pedestal_base" type="fixed">
+    <joint name="${prefix}hydra_base-rob2_base_link" type="fixed">
       <parent link="${prefix}hydra_base"/>
-      <child  link="${prefix}rob2_pedestal_base"/>
-      <origin xyz="${radius} 0 0" rpy="0 0 ${pi}"/>
+      <child  link="${prefix}rob2_base_link"/>
+      <origin xyz="${rob2_base_xyz}" rpy="${rob2_base_rpy}"/>>
     </joint>
-    <joint name="${prefix}hydra_base-rob3_pedestal_base" type="fixed">
+    <joint name="${prefix}hydra_base-rob3_base_link" type="fixed">
       <parent link="${prefix}hydra_base"/>
-      <child  link="${prefix}rob3_pedestal_base"/>
-      <origin xyz="-${radius*sin(pi/6)} ${radius*cos(pi/6)} 0" rpy="0 0 -${pi/3}"/>
+      <child  link="${prefix}rob3_base_link"/>
+      <origin xyz="${rob3_base_xyz}" rpy="${rob3_base_rpy}"/>
     </joint>
-    <joint name="${prefix}hydra_base-$(arg prefix)rotary_table_base" type="fixed">
+    <joint name="${prefix}hydra_base-$(arg prefix)positioner_static" type="fixed">
       <parent link="${prefix}hydra_base"/>
-      <child  link="${prefix}positioner_stand_base"/>
-      <origin xyz="0 0 0"/>
+      <child  link="${prefix}positioner_static"/>
+      <origin xyz="${wobj_xyz}" rpy="${wobj_rpy}"/>
     </joint>
   </xacro:macro>

File: urdf/positioner/positioner.xacro (robot description, xacro)
@@ -4,8 +4,8 @@
   <xacro:include filename="$(find hydra_description)/urdf/positioner/positioner_macro.xacro"/>
   <xacro:positioner_macro prefix="$(arg prefix)"/>
-  <link name="world" />
+  <link name="world"/>
   <joint name="world-$(arg prefix)hydra_positioner" type="fixed">
     <parent link="world"/>
-    <child link="$(arg prefix)positioner_stand_base"/>
+    <child link="$(arg prefix)positioner_static"/>
   </joint>
 </robot>

File: urdf/positioner/positioner_macro.xacro (robot description, xacro)
@@ -1,5 +1,5 @@
 <?xml version="1.0"?>
 <robot xmlns:xacro="http://www.ros.org/wiki/xacro">
-  <xacro:property name="pos_stand_height" value="0.32853" />
+  <xacro:property name="pos_stand_height" value="0.32853"/>
   <xacro:macro name="positioner_macro" params="prefix">
     <!-- link list -->
@@ -44,13 +44,8 @@
     <link name="${prefix}positioner_static"/>
     <!-- joint list -->
-    <joint name="${prefix}pos_stand_base-rotary_table_base" type="fixed">
-      <parent link="${prefix}positioner_stand_base"/>
-      <child link="${prefix}rotary_table_base"/>
-      <origin rpy="0.0 0.0 0.0" xyz="0 0 ${pos_stand_height}"/>
-    </joint>
-    <joint name="${prefix}rotary_table_top_base" type="fixed">
-      <parent link="${prefix}rotary_table_base"/>
-      <child link="${prefix}rotary_table_top"/>
-      <origin rpy="0.0 0.0 0.0" xyz="0 0 0.183984"/>
+    <joint name="${prefix}positioner_static_joint" type="fixed">
+      <parent link="${prefix}positioner_static"/>
+      <child  link="${prefix}rotary_table_top"/>
+      <origin rpy="0.0 0.0 0.0" xyz="0 0 -0.03175"/>
     </joint>
     <joint name="${prefix}positioner_joint" type="continuous">
@@ -63,11 +58,16 @@
     <joint name="${prefix}positioner_tcp_joint" type="fixed">
       <parent link="${prefix}positioner_base"/>
-      <child link="${prefix}positioner"/>
+      <child  link="${prefix}positioner"/>
       <origin rpy="0.0 0.0 0.0" xyz="0 0 0.03175"/>
     </joint>
-    <joint name="${prefix}positioner_static_joint" type="fixed">
+    <joint name="${prefix}rotary_table_top-${prefix}rotary_table_base" type="fixed">
       <parent link="${prefix}rotary_table_top"/>
-      <child link="${prefix}positioner_static"/>
-      <origin rpy="0.0 0.0 0.0" xyz="0 0 0.03175"/>
+      <child  link="${prefix}rotary_table_base"/>
+      <origin rpy="0.0 0.0 0.0" xyz="0 0 -0.183984"/>
+      </joint>
+    <joint name="${prefix}rotary_table_base-${prefix}pos_stand_base" type="fixed">
+      <parent link="${prefix}rotary_table_base"/>
+      <child  link="${prefix}positioner_stand_base"/>
+      <origin rpy="0.0 0.0 0.0" xyz="0 0 ${-pos_stand_height}"/>
     </joint>
   </xacro:macro>

File: urdf/robots/za_pedestal.xacro (robot description, xacro)
@@ -1,7 +1,15 @@
 <?xml version="1.0" ?>
 <robot name="za" xmlns:xacro="http://www.ros.org/wiki/xacro">
-  <xacro:arg name="prefix" default="" />
-  <xacro:arg name="tool" default="typhoon_extruder" />
-  <xacro:include filename="$(find hydra_description)/urdf/robots/za_pedestal_macro.xacro" />
-  <xacro:za_pedestal_macro prefix="$(arg prefix)" tool="$(arg tool)"/>
+  <xacro:arg name="prefix" default=""/>
+  <xacro:arg name="tool" default="typhoon_extruder"/>
+  <xacro:property name="tool_parameters_file" value="$(find hydra_description)/config/tool_parameters.yaml"/>
+  <xacro:property name="tool_data" value="${xacro.load_yaml(tool_parameters_file)}"/>
+  <xacro:include filename="$(find hydra_description)/urdf/robots/za_pedestal_macro.xacro"/>
+  <xacro:za_pedestal_macro prefix="$(arg prefix)" tool_data="${tool_data['rob1']}" tool="$(arg tool)"/>
+  <!-- 'world' frame: default pose reference frame -->
+  <link name="world"/>
+  <joint name="world-$(arg prefix)base_link" type="fixed">
+    <parent link="world"/>
+    <child link="$(arg prefix)base_link"/>
+  </joint>
 </robot>

File: urdf/robots/za_pedestal_macro.xacro (robot description, xacro)
@@ -1,8 +1,8 @@
 <?xml version="1.0"?>
 <robot xmlns:xacro="http://www.ros.org/wiki/xacro">
-  <xacro:property name="ped_height" value="0.585" />
-  <xacro:macro name="za_pedestal_macro" params="prefix tool:='tool0'" >
-    <xacro:include filename="$(find hydra_description)/urdf/robots/za_tool_macro.xacro" />
-    <xacro:za_tool_macro prefix="${prefix}" tool="${tool}"/>
+  <xacro:property name="ped_height" value="0.585"/>
+  <xacro:macro name="za_pedestal_macro" params="prefix tool_data tool:='tool0'" >
+    <xacro:include filename="$(find hydra_description)/urdf/robots/za_tool_macro.xacro"/>
+    <xacro:za_tool_macro prefix="${prefix}" tool_data="${tool_data}" tool="${tool}"/>
     <!-- link list -->
     <link name="${prefix}pedestal_base">
@@ -20,12 +20,12 @@
     <link name="${prefix}pedestal_top"/>
     <!-- joint list -->
-    <joint name="${prefix}pedestal_base-${prefix}pedestal_top" type="fixed">
-      <parent link="${prefix}pedestal_base"/>
+    <joint name="${prefix}base_link-${prefix}pedestal_top" type="fixed">
+      <parent link="${prefix}base_link"/>
       <child  link="${prefix}pedestal_top"/>
-      <origin rpy="0.0 0.0 0.0" xyz="0 0 ${ped_height}"/>
     </joint>
-    <joint name="${prefix}pedestal_top-${prefix}base_link" type="fixed">
+    <joint name="${prefix}pedestal_top-${prefix}pedestal_base" type="fixed">
       <parent link="${prefix}pedestal_top"/>
-      <child  link="${prefix}base_link"/>
+      <child  link="${prefix}pedestal_base"/>
+      <origin rpy="0.0 0.0 0.0" xyz="0 0 ${-ped_height}"/>
     </joint>
   </xacro:macro>

File: urdf/robots/za_tool.xacro (robot description, xacro)
@@ -1,15 +1,15 @@
 <?xml version="1.0" ?>
 <robot name="za" xmlns:xacro="http://www.ros.org/wiki/xacro">
-  <xacro:arg name="prefix" default="" />
-  <xacro:arg name="tool" default="typhoon_extruder" />
-  <xacro:include filename="$(find hydra_description)/urdf/robots/za_tool_macro.xacro" />
-  <xacro:za_tool_macro prefix="$(arg prefix)" tool="$(arg tool)"/>
+  <xacro:arg name="prefix" default=""/>
+  <xacro:arg name="tool" default="typhoon_extruder"/>
+  <xacro:property name="tool_parameters_file" value="$(find hydra_description)/config/tool_parameters.yaml"/>
+  <xacro:property name="tool_data" value="${xacro.load_yaml(tool_parameters_file)}"/>
+  <xacro:include filename="$(find hydra_description)/urdf/robots/za_tool_macro.xacro"/>
+  <xacro:za_tool_macro prefix="$(arg prefix)" tool_data="${tool_data['rob1']}" tool="$(arg tool)"/>
   <!-- 'world' frame: default pose reference frame -->
-  <link name="world" />
+  <link name="world"/>
   <joint name="world-$(arg prefix)base_link" type="fixed">
     <parent link="world"/>
     <child link="$(arg prefix)base_link"/>
-    <origin xyz="0 0 0" rpy="0 0 0"/>
-    <axis xyz="0 0 1"/>
   </joint>
 </robot>

File: urdf/robots/za_tool_macro.xacro (robot description, xacro)
@@ -1,11 +1,11 @@
 <?xml version="1.0"?>
 <robot xmlns:xacro="http://www.ros.org/wiki/xacro">
-  <xacro:macro name="za_tool_macro" params="prefix tool:='tool0'" >
-    <xacro:include filename="$(find za_description)/urdf/za_macro.xacro" />
-    <xacro:za_macro prefix="${prefix}" />
+  <xacro:macro name="za_tool_macro" params="prefix tool_data tool:='tool0'" >
+    <xacro:include filename="$(find za_description)/urdf/za_macro.xacro"/>
+    <xacro:za_macro prefix="${prefix}"/>
     <xml:property name="var" value="typhoon_extruder"/>
     <xacro:if value="${tool == 'typhoon_extruder'}">
-      <xacro:include filename="$(find hydra_description)/urdf/tools/typhoon_extruder_macro.xacro" />
-      <xacro:typhoon_extruder_macro prefix="${prefix}" />
+      <xacro:include filename="$(find hydra_description)/urdf/tools/typhoon_extruder_macro.xacro"/>
+      <xacro:typhoon_extruder_macro prefix="${prefix}" tool_data="${tool_data['typhoon_extruder']}"/>
     </xacro:if>
   </xacro:macro>

File: urdf/tools/typhoon_extruder_macro.xacro (robot description, xacro)
@@ -1,7 +1,7 @@
 <?xml version="1.0"?>
 <robot xmlns:xacro="http://www.ros.org/wiki/xacro">
-  <xacro:property name="tcp_trans" value="0.08613 0.0 -0.159" />
-  <xacro:property name="tcp_rot"  value="0.0 ${pi} 0.0" />
-  <xacro:macro name="typhoon_extruder_macro" params="prefix">
+  <xacro:macro name="typhoon_extruder_macro" params="prefix tool_data">
+    <xacro:property name="tcp_xyz" value="${tool_data['x']} ${tool_data['y']} ${tool_data['z']}"/>
+    <xacro:property name="tcp_rpy" value="${tool_data['roll']} ${tool_data['pitch']} ${tool_data['yaw']}"/>
     <!-- link list -->
     <link name="${prefix}typhoon_extruder">
@@ -16,21 +16,16 @@
         </geometry>
       </collision>
-      <inertial>
-          <origin xyz="0.065346 0.000016 -0.031645"/>
-          <mass value="1.75"/>
-        <inertia ixx="0.006265" ixy="0.000003" ixz="-0.000805" iyy="0.006649" iyz="0.000002" izz="0.001704"/>
-      </inertial>
     </link>
-    <link name="${prefix}typhoon_extruder_tcp" />
+    <link name="${prefix}typhoon_extruder_tcp"/>
     <!-- attach extruder to flange -->
     <joint name="${prefix}extruder_attach_joint" type="fixed">
       <parent link="${prefix}flange"/>
       <child link="${prefix}typhoon_extruder"/>
-      <origin xyz="0 0 0" rpy="0 0 0" />
+      <origin xyz="0 0 0" rpy="0 0 0"/>
     </joint>
     <joint name="${prefix}extruder_extruder_base" type="fixed">
       <parent link="${prefix}typhoon_extruder"/>
       <child link="${prefix}typhoon_extruder_tcp"/>
-      <origin xyz="${tcp_trans}" rpy="${tcp_rot}" />
+      <origin xyz="${tcp_xyz}" rpy="${tcp_rpy}"/>
     </joint>
   </xacro:macro>

Commit message: add missing rob3 mock hardware

File: urdf/hydra.xacro (robot description, xacro)
@@ -26,4 +26,7 @@
     <xacro:za_ros2_control prefix="$(arg prefix)rob1_" use_mock_hardware="$(arg use_mock_hardware)"/>
     <xacro:za_ros2_control prefix="$(arg prefix)rob2_" use_mock_hardware="$(arg use_mock_hardware)"/>
+    <xacro:za_ros2_control prefix="$(arg prefix)rob3_" use_mock_hardware="$(arg use_mock_hardware)"/>
+    <xacro:include filename="$(find hydra_description)/urdf/positioner/positioner.ros2_control.xacro"/>
+    <xacro:positioner_ros2_control prefix="$(arg prefix)" use_mock_hardware="$(arg use_mock_hardware)"/>
   </xacro:if>
 </robot>

File: urdf/hydra_macro.xacro (robot description, xacro)
@@ -46,5 +46,5 @@
       <origin xyz="${rob3_base_xyz}" rpy="${rob3_base_rpy}"/>
     </joint>
-    <joint name="${prefix}hydra_base-$(arg prefix)positioner_static" type="fixed">
+    <joint name="${prefix}hydra_base-${prefix}positioner_static" type="fixed">
       <parent link="${prefix}hydra_base"/>
       <child  link="${prefix}positioner_static"/>

File: urdf/positioner/positioner.ros2_control.xacro (robot description, xacro)
@@ -1,6 +1,6 @@
 <?xml version="1.0"?>
 <robot xmlns:xacro="http://www.ros.org/wiki/xacro">
-  <xacro:macro name="positioner_ros2_control" params="prefix use_mock_hardware:=^|true">
-    <ros2_control name="${prefix}ros2_control" type="system">
+  <xacro:macro name="positioner_ros2_control" params="prefix use_mock_hardware:=true">
+    <ros2_control name="${prefix}positioner_ros2_control" type="system">
       <hardware>
         <xacro:if value="${use_mock_hardware}">
