Commit message: feat: integrate urdf from za6_description package

File: urdf/hydra.xacro (robot description, xacro)
@@ -3,9 +3,11 @@
   <xacro:arg name="prefix" default=""/>
   <xacro:arg name="tool" default="typhoon_extruder"/>
-  <!-- ros2_control parameters-->
+  <xacro:arg name="include_ros2_control" default="false"/>
+  <xacro:arg name="ros2_control_name" default="hal_hw_interface"/>
   <xacro:arg name="use_mock_hardware" default="true"/>
-  <xacro:arg name="include_hardware" default="true"/>
+  <xacro:arg name="ros2_control_plugin"
+             default="hal_system_interface/HalSystemInterface"/>
   <xacro:arg name="initial_positions_file"
-    default="$(find hydra_description)/config/initial_positions.yaml"/>
+             default="$(find hydra_description)/config/initial_positions.yaml"/>
   <xacro:property name="tool_parameters_file" value="$(find hydra_description)/config/tool_parameters.yaml"/>
   <xacro:property name="kinematic_parameters_file" value="$(find hydra_description)/config/kinematic_parameters.yaml"/>
@@ -19,22 +21,31 @@
     rob3_tool="$(arg tool)"
   />
+  <xacro:if value="$(arg include_ros2_control)">
+    <xacro:include filename="$(find za6_description)/urdf/za6.ros2_control.xacro"/>
+    <xacro:za6_ros2_control
+      name="$(arg ros2_control_name)"
+      prefix="$(arg prefix)rob1_"
+      use_mock_hardware="$(arg use_mock_hardware)"
+      initial_positions_file="$(arg initial_positions_file)"
+      ros2_control_plugin="$(arg ros2_control_plugin)"/>
+    <xacro:za6_ros2_control
+      name="$(arg ros2_control_name)"
+      prefix="$(arg prefix)rob2_"
+      use_mock_hardware="$(arg use_mock_hardware)"
+      initial_positions_file="$(arg initial_positions_file)"
+      ros2_control_plugin="$(arg ros2_control_plugin)"/>
+    <xacro:za6_ros2_control
+      name="$(arg ros2_control_name)"
+      prefix="$(arg prefix)rob3_"
+      use_mock_hardware="$(arg use_mock_hardware)"
+      initial_positions_file="$(arg initial_positions_file)"
+      ros2_control_plugin="$(arg ros2_control_plugin)"/>
+    <xacro:include filename="$(find hydra_description)/urdf/positioner/positioner.ros2_control.xacro"/>
+    <xacro:positioner_ros2_control prefix="$(arg prefix)" use_mock_hardware="$(arg use_mock_hardware)"/>
+  </xacro:if>
   <link name="world"/>
   <joint name="world-$(arg prefix)hydra_base" type="fixed">
     <parent link="world"/>
-    <child  link="$(arg prefix)hydra_base"/>
+    <child link="$(arg prefix)hydra_base"/>
   </joint>
-  <xacro:if value="$(arg include_hardware)">
-    <xacro:include filename="$(find za_description)/urdf/za.ros2_control.xacro"/>
-    <xacro:za_ros2_control prefix="$(arg prefix)rob1_"
-      use_mock_hardware="$(arg use_mock_hardware)"
-      initial_positions_file="$(arg initial_positions_file)"/>
-    <xacro:za_ros2_control prefix="$(arg prefix)rob2_"
-      use_mock_hardware="$(arg use_mock_hardware)"
-      initial_positions_file="$(arg initial_positions_file)"/>
-    <xacro:za_ros2_control prefix="$(arg prefix)rob3_"
-      use_mock_hardware="$(arg use_mock_hardware)"
-      initial_positions_file="$(arg initial_positions_file)"/>
-    <xacro:include filename="$(find hydra_description)/urdf/positioner/positioner.ros2_control.xacro"/>
-    <xacro:positioner_ros2_control prefix="$(arg prefix)" use_mock_hardware="$(arg use_mock_hardware)"/>
-  </xacro:if>
 </robot>

File: urdf/hydra_macro.xacro (robot description, xacro)
@@ -1,5 +1,5 @@
 <?xml version="1.0" ?>
 <robot name="hydra" xmlns:xacro="http://www.ros.org/wiki/xacro">
-  <xacro:include filename="$(find hydra_description)/urdf/robots/za_pedestal_macro.xacro"/>
+  <xacro:include filename="$(find hydra_description)/urdf/robots/za6_pedestal_macro.xacro"/>
   <xacro:include filename="$(find hydra_description)/urdf/positioner/positioner_macro.xacro"/>
   <xacro:macro name="hydra_macro" params="
@@ -26,7 +26,7 @@
     <xacro:property name="rob3_base_xyz" value="${rob3_base_data['x']} ${rob3_base_data['y']} ${rob3_base_data['z']}"/>
     <xacro:property name="rob3_base_rpy" value="${rob3_base_data['roll']} ${rob3_base_data['pitch']} ${rob3_base_data['yaw']}"/>
-    <xacro:za_pedestal_macro prefix="${prefix}rob1_" tool_data="${tool_data['rob1']}" tool="${rob1_tool}"/>
-    <xacro:za_pedestal_macro prefix="${prefix}rob2_" tool_data="${tool_data['rob2']}" tool="${rob2_tool}"/>
-    <xacro:za_pedestal_macro prefix="${prefix}rob3_" tool_data="${tool_data['rob3']}" tool="${rob3_tool}"/>
+    <xacro:za6_pedestal_macro prefix="${prefix}rob1_" tool_data="${tool_data['rob1']}" tool="${rob1_tool}"/>
+    <xacro:za6_pedestal_macro prefix="${prefix}rob2_" tool_data="${tool_data['rob2']}" tool="${rob2_tool}"/>
+    <xacro:za6_pedestal_macro prefix="${prefix}rob3_" tool_data="${tool_data['rob3']}" tool="${rob3_tool}"/>
     <xacro:positioner_macro prefix="${prefix}"/>
     <link name="${prefix}hydra_base"/>

File: urdf/robots/za6_pedestal.xacro (robot description, xacro)
@@ -8,6 +8,6 @@
   <xacro:property name="tool_parameters_file" value="$(find hydra_description)/config/tool_parameters.yaml"/>
   <xacro:property name="tool_data" value="${xacro.load_yaml(tool_parameters_file)}"/>
-  <xacro:include filename="$(find hydra_description)/urdf/robots/za_pedestal_macro.xacro"/>
-  <xacro:za_pedestal_macro prefix="$(arg prefix)" tool_data="${tool_data['rob1']}" tool="$(arg tool)"/>
+  <xacro:include filename="$(find hydra_description)/urdf/robots/za6_pedestal_macro.xacro"/>
+  <xacro:za6_pedestal_macro prefix="$(arg prefix)" tool_data="${tool_data['rob1']}" tool="$(arg tool)"/>
   <!-- 'world' frame - default pose reference frame -->
   <link name="world"/>
@@ -17,6 +17,6 @@
   </joint>
   <xacro:if value="$(arg include_hardware)">
-    <xacro:include filename="$(find za_description)/urdf/za.ros2_control.xacro"/>
-    <xacro:za_ros2_control prefix="$(arg prefix)" use_mock_hardware="$(arg use_mock_hardware)"/>
+    <xacro:include filename="$(find za6_description)/urdf/za6.ros2_control.xacro"/>
+    <xacro:za6_ros2_control prefix="$(arg prefix)" use_mock_hardware="$(arg use_mock_hardware)"/>
   </xacro:if>
 </robot>

File: urdf/robots/za6_pedestal_macro.xacro (robot description, xacro)
@@ -2,17 +2,17 @@
 <robot xmlns:xacro="http://www.ros.org/wiki/xacro">
   <xacro:property name="ped_height" value="0.585"/>
-  <xacro:macro name="za_pedestal_macro" params="prefix tool_data tool:='tool0'" >
-    <xacro:include filename="$(find hydra_description)/urdf/robots/za_tool_macro.xacro"/>
-    <xacro:za_tool_macro prefix="${prefix}" tool_data="${tool_data}" tool="${tool}"/>
+  <xacro:macro name="za6_pedestal_macro" params="prefix tool_data tool:='tool0'" >
+    <xacro:include filename="$(find hydra_description)/urdf/robots/za6_tool_macro.xacro"/>
+    <xacro:za6_tool_macro prefix="${prefix}" tool_data="${tool_data}" tool="${tool}"/>
     <!-- link list -->
     <link name="${prefix}pedestal_base">
       <visual>
         <geometry>
-          <mesh filename="package://hydra_description/meshes/visual/za_pedestal.dae"/>
+          <mesh filename="package://hydra_description/meshes/visual/za6_pedestal.dae"/>
         </geometry>
       </visual>
       <collision>
         <geometry>
-          <mesh filename="package://hydra_description/meshes/collision/za_pedestal_collision.stl"/>
+          <mesh filename="package://hydra_description/meshes/collision/za6_pedestal_collision.stl"/>
         </geometry>
       </collision>

File: urdf/robots/za6_tool.xacro (robot description, xacro)
@@ -12,6 +12,6 @@
   <xacro:property name="tool_parameters_file" value="$(find hydra_description)/config/tool_parameters.yaml"/>
   <xacro:property name="tool_data" value="${xacro.load_yaml(tool_parameters_file)}"/>
-  <xacro:include filename="$(find hydra_description)/urdf/robots/za_tool_macro.xacro"/>
-  <xacro:za_tool_macro prefix="$(arg prefix)" tool_data="${tool_data['rob1']}" tool="$(arg tool)"/>
+  <xacro:include filename="$(find hydra_description)/urdf/robots/za6_tool_macro.xacro"/>
+  <xacro:za6_tool_macro prefix="$(arg prefix)" tool_data="${tool_data['rob1']}" tool="$(arg tool)"/>
   <!-- 'world' frame - default pose reference frame -->
   <link name="world"/>
@@ -21,6 +21,6 @@
   </joint>
   <xacro:if value="$(arg include_hardware)">
-    <xacro:include filename="$(find za_description)/urdf/za.ros2_control.xacro"/>
-    <xacro:za_ros2_control prefix="$(arg prefix)"
+    <xacro:include filename="$(find za6_description)/urdf/za6.ros2_control.xacro"/>
+    <xacro:za6_ros2_control prefix="$(arg prefix)"
       use_mock_hardware="$(arg use_mock_hardware)"
       initial_positions_file="$(arg initial_positions_file)"/>

File: urdf/robots/za6_tool_macro.xacro (robot description, xacro)
@@ -1,7 +1,7 @@
 <?xml version="1.0"?>
 <robot xmlns:xacro="http://www.ros.org/wiki/xacro">
-  <xacro:macro name="za_tool_macro" params="prefix tool_data tool:='tool0'" >
-    <xacro:include filename="$(find za_description)/urdf/za_macro.xacro"/>
-    <xacro:za_macro prefix="${prefix}"/>
+  <xacro:macro name="za6_tool_macro" params="prefix tool_data tool:='tool0'" >
+    <xacro:include filename="$(find za6_description)/urdf/za6_macro.xacro"/>
+    <xacro:za6 prefix="${prefix}" tool0_trans="0 0 0" tool0_rot="0 0 0"/>
     <xml:property name="var" value="typhoon_extruder"/>
     <xacro:if value="${tool == 'typhoon_extruder'}">

File: urdf/tools/typhoon_extruder_macro.xacro (robot description, xacro)
@@ -22,8 +22,8 @@
       <parent link="${prefix}flange"/>
       <child link="${prefix}typhoon_extruder"/>
-      <origin xyz="0 0 0" rpy="0 0 0"/>
+      <origin xyz="0 0 0" rpy="${pi} ${-pi/2} 0"/>
     </joint>
-    <joint name="${prefix}extruder_extruder_base" type="fixed">
-      <parent link="${prefix}typhoon_extruder"/>
+    <joint name="${prefix}flange-extruder_tcp" type="fixed">
+      <parent link="${prefix}flange"/>
       <child link="${prefix}typhoon_extruder_tcp"/>
       <origin xyz="${tcp_xyz}" rpy="${tcp_rpy}"/>
