Commit message: update hydra_ros to be compatible with kintrol library

File: urdf/positioner/positioner_macro.xacro (robot description, xacro)
@@ -59,4 +59,5 @@
       <parent link="${prefix}rotary_table_top"/>
       <child link="${prefix}positioner_base"/>
+      <limit effort="1000.0" velocity="1.5"/>
     </joint>
     <joint name="${prefix}positioner_joint" type="fixed">

Commit message: add positioner_state_controller

File: urdf/positioner/positioner_macro.xacro (robot description, xacro)
@@ -4,4 +4,6 @@
   <xacro:include filename="$(find za_description)/urdf/utils.xacro"/>
   <xacro:macro name="positioner_macro" params="prefix">
+    <!-- Is the robot being simulated in gazebo?" -->
+    <xacro:arg name="gazebo" default="true" />
     <!-- link list -->
     <link name="${prefix}positioner_stand_base">
@@ -64,5 +66,6 @@
       <child link="${prefix}rotary_table_top"/>
     </joint>
-    <joint name="${prefix}rotary_table_positioner" type="continuous">
+    <joint name="${prefix}positioner_joint" type="continuous">
+    <!--<joint name="${prefix}rotary_table_positioner" type="continuous">-->
       <origin rpy="0.0 0.0 0.0" xyz="0 0 0"/>
       <axis xyz="0 0 1"/>
@@ -71,5 +74,5 @@
       <limit effort="1000.0" velocity="1.5"/>
     </joint>
-    <joint name="${prefix}positioner_joint" type="fixed">
+    <joint name="${prefix}positioner_tcp_joint" type="fixed">
       <origin rpy="0.0 0.0 0.0" xyz="0 0 0.03175"/>
       <parent link="${prefix}positioner_base"/>
@@ -81,5 +84,15 @@
       <child link="${prefix}positioner_static"/>
     </joint>
-    <xacro:gazebo-joint joint="${prefix}rotary_table_positioner" transmission="hardware_interface/VelocityJointInterface"/>
+    <!-- Define additional Gazebo tags -->
+    <xacro:if value="$(arg gazebo)">
+      <xacro:gazebo-joint joint="${prefix}positioner_joint" transmission="hardware_interface/EffortJointInterface"/>
+      <xacro:gazebo-joint joint="${prefix}positioner_joint" transmission="hardware_interface/VelocityJointInterface"/>
+      <xacro:gazebo-joint joint="${prefix}positioner_joint" transmission="hardware_interface/PositionJointInterface"/>
+      <transmission name="${prefix}positioner_state">
+        <type>hydra_hw/PositionerStateInterface</type>
+        <joint name="${prefix}positioner_joint"><hardwareInterface>hydra_hw/PositionerStateInterface</hardwareInterface></joint>
+        <actuator name="${prefix}positioner_motor"><hardwareInterface>hydra_hw/PositionerStateInterface</hardwareInterface></actuator>
+      </transmission>
+    </xacro:if>
   </xacro:macro>
 </robot>

Commit message: fix formatting and includes in urdf

File: urdf/positioner/positioner_macro.xacro (robot description, xacro)
@@ -2,5 +2,4 @@
 <robot xmlns:xacro="http://www.ros.org/wiki/xacro">
   <xacro:property name="pos_stand_height" value="0.32853" />
-  <xacro:include filename="$(find za_description)/urdf/utils.xacro"/>
   <xacro:macro name="positioner_macro" params="prefix">
     <!-- link list -->
@@ -16,5 +15,4 @@
         </geometry>
       </collision>
-      <xacro:default_inertial mass="1"/>
     </link>
     <link name="${prefix}rotary_table_base">
@@ -29,9 +27,6 @@
         </geometry>
       </collision>
-      <xacro:default_inertial mass="1"/>
     </link>
-    <link name="${prefix}rotary_table_top">
-      <xacro:default_inertial mass="1"/>
-    </link>
+    <link name="${prefix}rotary_table_top"/>
     <link name="${prefix}positioner_base">
       <visual>
@@ -45,9 +40,4 @@
         </geometry>
       </collision>
-      <inertial>
-        <origin xyz="0.000000 0.000000 0.006349"/>
-        <mass value="27.67"/>
-        <inertia ixx="1.929232" ixy="0.000000" ixz="0.000000" iyy="1.929232" iyz="0.000000" izz="3.857721"/>
-      </inertial>
     </link>
     <link name="${prefix}positioner"/>
@@ -55,29 +45,29 @@
     <!-- joint list -->
     <joint name="${prefix}pos_stand_base-rotary_table_base" type="fixed">
-      <origin rpy="0.0 0.0 0.0" xyz="0 0 ${pos_stand_height}"/>
       <parent link="${prefix}positioner_stand_base"/>
       <child link="${prefix}rotary_table_base"/>
+      <origin rpy="0.0 0.0 0.0" xyz="0 0 ${pos_stand_height}"/>
     </joint>
     <joint name="${prefix}rotary_table_top_base" type="fixed">
-      <origin rpy="0.0 0.0 0.0" xyz="0 0 0.183984"/>
       <parent link="${prefix}rotary_table_base"/>
       <child link="${prefix}rotary_table_top"/>
+      <origin rpy="0.0 0.0 0.0" xyz="0 0 0.183984"/>
     </joint>
     <joint name="${prefix}positioner_joint" type="continuous">
+      <parent link="${prefix}rotary_table_top"/>
+      <child link="${prefix}positioner_base"/>
       <origin rpy="0.0 0.0 0.0" xyz="0 0 0"/>
       <axis xyz="0 0 1"/>
-      <parent link="${prefix}rotary_table_top"/>
-      <child link="${prefix}positioner_base"/>
-      <limit effort="1000.0" velocity="1.5"/>
+      <limit effort="0" velocity="1.5"/>
     </joint>
     <joint name="${prefix}positioner_tcp_joint" type="fixed">
-      <origin rpy="0.0 0.0 0.0" xyz="0 0 0.03175"/>
       <parent link="${prefix}positioner_base"/>
       <child link="${prefix}positioner"/>
+      <origin rpy="0.0 0.0 0.0" xyz="0 0 0.03175"/>
     </joint>
     <joint name="${prefix}positioner_static_joint" type="fixed">
-      <origin rpy="0.0 0.0 0.0" xyz="0 0 0.03175"/>
       <parent link="${prefix}rotary_table_top"/>
       <child link="${prefix}positioner_static"/>
+      <origin rpy="0.0 0.0 0.0" xyz="0 0 0.03175"/>
     </joint>
   </xacro:macro>

File: urdf/robots/za_pedestal_macro.xacro (robot description, xacro)
@@ -2,7 +2,7 @@
 <robot xmlns:xacro="http://www.ros.org/wiki/xacro">
   <xacro:property name="ped_height" value="0.585" />
-	<xacro:macro name="za_pedestal_macro" params="prefix tool:='tool0'" >
-		<xacro:include filename="$(find hydra_description)/urdf/robots/za_tool_macro.xacro" />
-		<xacro:za_tool_macro prefix="${prefix}" tool="${tool}"/>
+  <xacro:macro name="za_pedestal_macro" params="prefix tool:='tool0'" >
+    <xacro:include filename="$(find hydra_description)/urdf/robots/za_tool_macro.xacro" />
+    <xacro:za_tool_macro prefix="${prefix}" tool="${tool}"/>
     <link name="${prefix}pedestal_base">
       <visual>
@@ -17,5 +17,5 @@
       </collision>
     </link>
-		<link name="${prefix}pedestal_top"/>
+    <link name="${prefix}pedestal_top"/>
     <joint name="${prefix}pedestal_base-${prefix}pedestal_top" type="fixed">
       <origin rpy="0.0 0.0 0.0" xyz="0 0 ${ped_height}"/>
@@ -27,4 +27,4 @@
       <child  link="${prefix}base_link"/>
     </joint>
-	</xacro:macro>
+  </xacro:macro>
 </robot>

File: urdf/robots/za_tool_macro.xacro (robot description, xacro)
@@ -1,12 +1,12 @@
 <?xml version="1.0"?>
 <robot xmlns:xacro="http://www.ros.org/wiki/xacro">
-	<xacro:macro name="za_tool_macro" params="prefix tool:='tool0'" >
-		<xacro:include filename="$(find za_description)/urdf/za_macro.xacro" />
-		<xacro:za_macro prefix="${prefix}"/>
-		<xml:property name="var" value="typhoon_extruder"/>
-		<xacro:if value="${tool == 'typhoon_extruder'}">
-			<xacro:include filename="$(find hydra_description)/urdf/tools/typhoon_extruder_macro.xacro" />
-			<xacro:typhoon_extruder_macro prefix="${prefix}" />
-		</xacro:if>
+  <xacro:macro name="za_tool_macro" params="prefix tool:='tool0'" >
+    <xacro:include filename="$(find za_description)/urdf/za_macro.xacro" />
+    <xacro:za_macro prefix="${prefix}"/>
+    <xml:property name="var" value="typhoon_extruder"/>
+    <xacro:if value="${tool == 'typhoon_extruder'}">
+      <xacro:include filename="$(find hydra_description)/urdf/tools/typhoon_extruder_macro.xacro" />
+      <xacro:typhoon_extruder_macro prefix="${prefix}" />
+    </xacro:if>
   </xacro:macro>
 </robot>

File: urdf/tools/typhoon_extruder_macro.xacro (robot description, xacro)
@@ -1,37 +1,37 @@
 <?xml version="1.0"?>
 <robot xmlns:xacro="http://www.ros.org/wiki/xacro">
-    <xacro:property name="tcp_trans" value="0.08613 0.0 -0.159" />
-    <xacro:property name="tcp_rot"  value="0.0 ${pi} 0.0" />
-	<xacro:macro name="typhoon_extruder_macro" params="prefix">
-		<!-- link list -->
-		<link name="${prefix}typhoon_extruder">
-			<visual>
-				<geometry>
-					<mesh filename="package://hydra_description/meshes/visual/typhoon_extruder.dae"/>
-				</geometry>
-			</visual>
-			<collision>
-				<geometry>
-					<mesh filename="package://hydra_description/meshes/collision/typhoon_extruder_collision.stl"/>
-				</geometry>
-			</collision>
-			<inertial>
-    			<origin xyz="0.065346 0.000016 -0.031645"/>
-    			<mass value="1.75"/>
-				<inertia ixx="0.006265" ixy="0.000003" ixz="-0.000805" iyy="0.006649" iyz="0.000002" izz="0.001704"/>
-			</inertial>
-		</link>
-		<link name="${prefix}typhoon_extruder_tcp" />
-		<!-- attach extruder to flange -->
-		<joint name="${prefix}extruder_attach_joint" type="fixed">
-			<origin xyz="0 0 0" rpy="0 0 0" />
-			<parent link="${prefix}flange"/>
-			<child link="${prefix}typhoon_extruder"/>
-		</joint>
-		<joint name="${prefix}extruder_extruder_base" type="fixed">
-			<origin xyz="${tcp_trans}" rpy="${tcp_rot}" />
-			<parent link="${prefix}typhoon_extruder"/>
-			<child link="${prefix}typhoon_extruder_tcp"/>
-		</joint>
-	</xacro:macro>
+  <xacro:property name="tcp_trans" value="0.08613 0.0 -0.159" />
+  <xacro:property name="tcp_rot"  value="0.0 ${pi} 0.0" />
+  <xacro:macro name="typhoon_extruder_macro" params="prefix">
+    <!-- link list -->
+    <link name="${prefix}typhoon_extruder">
+      <visual>
+        <geometry>
+          <mesh filename="package://hydra_description/meshes/visual/typhoon_extruder.dae"/>
+        </geometry>
+      </visual>
+      <collision>
+        <geometry>
+          <mesh filename="package://hydra_description/meshes/collision/typhoon_extruder_collision.stl"/>
+        </geometry>
+      </collision>
+      <inertial>
+          <origin xyz="0.065346 0.000016 -0.031645"/>
+          <mass value="1.75"/>
+        <inertia ixx="0.006265" ixy="0.000003" ixz="-0.000805" iyy="0.006649" iyz="0.000002" izz="0.001704"/>
+      </inertial>
+    </link>
+    <link name="${prefix}typhoon_extruder_tcp" />
+    <!-- attach extruder to flange -->
+    <joint name="${prefix}extruder_attach_joint" type="fixed">
+      <origin xyz="0 0 0" rpy="0 0 0" />
+      <parent link="${prefix}flange"/>
+      <child link="${prefix}typhoon_extruder"/>
+    </joint>
+    <joint name="${prefix}extruder_extruder_base" type="fixed">
+      <origin xyz="${tcp_trans}" rpy="${tcp_rot}" />
+      <parent link="${prefix}typhoon_extruder"/>
+      <child link="${prefix}typhoon_extruder_tcp"/>
+    </joint>
+  </xacro:macro>
 </robot>
