Commit message: fix spacings in closing tags

File: urdf/positioner/positioner.xacro (robot description, xacro)
@@ -4,5 +4,5 @@
   <xacro:include filename="$(find hydra_description)/urdf/positioner/positioner_macro.xacro"/>
   <xacro:positioner_macro prefix="$(arg prefix)"/>
-  <link name="world" />
+  <link name="world"/>
   <joint name="world-$(arg prefix)hydra_positioner" type="fixed">
     <parent link="world"/>

File: urdf/positioner/positioner_macro.xacro (robot description, xacro)
@@ -1,5 +1,5 @@
 <?xml version="1.0"?>
 <robot xmlns:xacro="http://www.ros.org/wiki/xacro">
-  <xacro:property name="pos_stand_height" value="0.32853" />
+  <xacro:property name="pos_stand_height" value="0.32853"/>
   <xacro:macro name="positioner_macro" params="prefix">
     <!-- link list -->

File: urdf/robots/za_pedestal.xacro (robot description, xacro)
@@ -1,12 +1,12 @@
 <?xml version="1.0" ?>
 <robot name="za" xmlns:xacro="http://www.ros.org/wiki/xacro">
-  <xacro:arg name="prefix" default="" />
+  <xacro:arg name="prefix" default=""/>
   <xacro:arg name="tool" default="typhoon_extruder"/>
   <xacro:property name="tool_parameters_file" value="$(find hydra_description)/config/tool_parameters.yaml"/>
   <xacro:property name="tool_data" value="${xacro.load_yaml(tool_parameters_file)}"/>
-  <xacro:include filename="$(find hydra_description)/urdf/robots/za_pedestal_macro.xacro" />
+  <xacro:include filename="$(find hydra_description)/urdf/robots/za_pedestal_macro.xacro"/>
   <xacro:za_pedestal_macro prefix="$(arg prefix)" tool_data="${tool_data['rob1']}" tool="$(arg tool)"/>
   <!-- 'world' frame: default pose reference frame -->
-  <link name="world" />
+  <link name="world"/>
   <joint name="world-$(arg prefix)base_link" type="fixed">
     <parent link="world"/>

File: urdf/robots/za_tool.xacro (robot description, xacro)
@@ -1,12 +1,12 @@
 <?xml version="1.0" ?>
 <robot name="za" xmlns:xacro="http://www.ros.org/wiki/xacro">
-  <xacro:arg name="prefix" default="" />
+  <xacro:arg name="prefix" default=""/>
   <xacro:arg name="tool" default="typhoon_extruder"/>
   <xacro:property name="tool_parameters_file" value="$(find hydra_description)/config/tool_parameters.yaml"/>
   <xacro:property name="tool_data" value="${xacro.load_yaml(tool_parameters_file)}"/>
-  <xacro:include filename="$(find hydra_description)/urdf/robots/za_tool_macro.xacro" />
+  <xacro:include filename="$(find hydra_description)/urdf/robots/za_tool_macro.xacro"/>
   <xacro:za_tool_macro prefix="$(arg prefix)" tool_data="${tool_data['rob1']}" tool="$(arg tool)"/>
   <!-- 'world' frame: default pose reference frame -->
-  <link name="world" />
+  <link name="world"/>
   <joint name="world-$(arg prefix)base_link" type="fixed">
     <parent link="world"/>

File: urdf/robots/za_tool_macro.xacro (robot description, xacro)
@@ -2,12 +2,12 @@
 <robot xmlns:xacro="http://www.ros.org/wiki/xacro">
   <xacro:macro name="za_tool_macro" params="prefix tool_data tool:='tool0'">
-    <xacro:include filename="$(find za_description)/urdf/za_macro.xacro" />
+    <xacro:include filename="$(find za_description)/urdf/za_macro.xacro"/>
     <xacro:za_macro prefix="${prefix}"/>
     <xacro:if value="${tool == 'typhoon_extruder'}">
-      <xacro:include filename="$(find hydra_description)/urdf/tools/typhoon_extruder_macro.xacro" />
+      <xacro:include filename="$(find hydra_description)/urdf/tools/typhoon_extruder_macro.xacro"/>
       <xacro:typhoon_extruder_macro prefix="${prefix}" tool_data="${tool_data['typhoon_extruder']}"/>
     </xacro:if>
     <xacro:if value="${tool == 'marker_tool'}">
-      <xacro:include filename="$(find hydra_description)/urdf/tools/marker_tool_macro.xacro" />
+      <xacro:include filename="$(find hydra_description)/urdf/tools/marker_tool_macro.xacro"/>
       <xacro:marker_tool_macro prefix="${prefix}" tool_data="${tool_data['marker_tool']}"/>
     </xacro:if>

File: urdf/tools/marker_tool_macro.xacro (robot description, xacro)
@@ -17,10 +17,10 @@
       </collision>
     </link>
-    <link name="${prefix}marker_tool_tcp" />
+    <link name="${prefix}marker_tool_tcp"/>
     <!-- attach marker to flange -->
     <joint name="${prefix}marker_attach_joint" type="fixed">
       <parent link="${prefix}flange"/>
       <child link="${prefix}marker_tool"/>
-      <origin xyz="0 0 0" rpy="0 0 0" />
+      <origin xyz="0 0 0" rpy="0 0 0"/>
     </joint>
     <joint name="${prefix}marker_marker_base" type="fixed">

File: urdf/tools/typhoon_extruder_macro.xacro (robot description, xacro)
@@ -17,15 +17,15 @@
       </collision>
     </link>
-    <link name="${prefix}typhoon_extruder_tcp" />
+    <link name="${prefix}typhoon_extruder_tcp"/>
     <!-- attach extruder to flange -->
     <joint name="${prefix}extruder_attach_joint" type="fixed">
       <parent link="${prefix}flange"/>
       <child link="${prefix}typhoon_extruder"/>
-      <origin xyz="0 0 0" rpy="0 0 0" />
+      <origin xyz="0 0 0" rpy="0 0 0"/>
     </joint>
     <joint name="${prefix}extruder_extruder_base" type="fixed">
       <parent link="${prefix}typhoon_extruder"/>
       <child link="${prefix}typhoon_extruder_tcp"/>
-      <origin xyz="${tcp_xyz}" rpy="${tcp_rpy}" />
+      <origin xyz="${tcp_xyz}" rpy="${tcp_rpy}"/>
     </joint>
   </xacro:macro>
