Commit message: fix indentation and remove Gazebo tags

File: urdf/robots/za_pedestal_macro.xacro (robot description, xacro)
@@ -3,7 +3,7 @@
   <xacro:property name="ped_height" value="0.585"/>
   <xacro:property name="base_height" value="0.2"/>
-	<xacro:macro name="za_pedestal_macro" params="prefix tool:='tool0'" >
-		<xacro:include filename="$(find hydra_description)/urdf/robots/za_tool_macro.xacro" />
-		<xacro:za_tool_macro prefix="${prefix}" tool="${tool}"/>
+  <xacro:macro name="za_pedestal_macro" params="prefix tool:='tool0'" >
+    <xacro:include filename="$(find hydra_description)/urdf/robots/za_tool_macro.xacro" />
+    <xacro:za_tool_macro prefix="${prefix}" tool="${tool}"/>
     <link name="${prefix}pedestal_base">
       <visual>
@@ -30,5 +30,5 @@
       </collision>
     </link>
-		<link name="${prefix}pedestal_top"/>
+    <link name="${prefix}pedestal_top"/>
     <joint name="${prefix}pedestal_base-${prefix}pedestal" type="fixed">
       <origin rpy="0.0 0.0 0.0" xyz="0 0 ${base_height}"/>
@@ -45,4 +45,4 @@
       <child  link="${prefix}base_link"/>
     </joint>
-	</xacro:macro>
+  </xacro:macro>
 </robot>

File: urdf/tools/typhoon_extruder_macro.xacro (robot description, xacro)
@@ -3,35 +3,35 @@
   <xacro:property name="tcp_trans" value="0.08613 0.0 -0.159" />
   <xacro:property name="tcp_rot"  value="0.0 ${pi} 0.0" />
-	<xacro:macro name="typhoon_extruder_macro" params="prefix">
-		<!-- link list -->
-		<link name="${prefix}typhoon_extruder">
-			<visual>
-				<geometry>
-					<mesh filename="package://hydra_description/meshes/visual/typhoon_extruder.dae"/>
-				</geometry>
-			</visual>
-			<collision>
-				<geometry>
-					<mesh filename="package://hydra_description/meshes/collision/typhoon_extruder_collision.stl"/>
-				</geometry>
-			</collision>
-			<inertial>
-    			<origin xyz="0.065346 0.000016 -0.031645"/>
-    			<mass value="1.75"/>
-				<inertia ixx="0.006265" ixy="0.000003" ixz="-0.000805" iyy="0.006649" iyz="0.000002" izz="0.001704"/>
-			</inertial>
-		</link>
-		<link name="${prefix}typhoon_extruder_tcp" />
-		<!-- attach extruder to flange -->
-		<joint name="${prefix}extruder_attach_joint" type="fixed">
-			<origin xyz="0 0 0" rpy="0 0 0" />
-			<parent link="${prefix}flange"/>
-			<child link="${prefix}typhoon_extruder"/>
-		</joint>
-		<joint name="${prefix}extruder_extruder_base" type="fixed">
-			<origin xyz="${tcp_trans}" rpy="${tcp_rot}" />
-			<parent link="${prefix}typhoon_extruder"/>
-			<child link="${prefix}typhoon_extruder_tcp"/>
-		</joint>
-	</xacro:macro>
+  <xacro:macro name="typhoon_extruder_macro" params="prefix">
+    <!-- link list -->
+    <link name="${prefix}typhoon_extruder">
+      <visual>
+        <geometry>
+          <mesh filename="package://hydra_description/meshes/visual/typhoon_extruder.dae"/>
+        </geometry>
+      </visual>
+      <collision>
+        <geometry>
+          <mesh filename="package://hydra_description/meshes/collision/typhoon_extruder_collision.stl"/>
+        </geometry>
+      </collision>
+      <inertial>
+          <origin xyz="0.065346 0.000016 -0.031645"/>
+          <mass value="1.75"/>
+        <inertia ixx="0.006265" ixy="0.000003" ixz="-0.000805" iyy="0.006649" iyz="0.000002" izz="0.001704"/>
+      </inertial>
+    </link>
+    <link name="${prefix}typhoon_extruder_tcp" />
+    <!-- attach extruder to flange -->
+    <joint name="${prefix}extruder_attach_joint" type="fixed">
+      <origin xyz="0 0 0" rpy="0 0 0" />
+      <parent link="${prefix}flange"/>
+      <child link="${prefix}typhoon_extruder"/>
+    </joint>
+    <joint name="${prefix}extruder_extruder_base" type="fixed">
+      <origin xyz="${tcp_trans}" rpy="${tcp_rot}" />
+      <parent link="${prefix}typhoon_extruder"/>
+      <child link="${prefix}typhoon_extruder_tcp"/>
+    </joint>
+  </xacro:macro>
 </robot>
